File: Work_in_progress/tools/Schematics/myth.kicad_sch (KiCad schematic)
At the start: 129 parts, among them J1 Conn_01x08_Male, J2 Conn_01x08_Male, J3 Conn_01x08_Male, J4 Conn_01x08_Male, J5 Conn_01x04_Male, J6 Conn_01x04_Male, J7 Conn_02x01, U1 74AHC02, U10 74HC238, U11 74HC238, U12 74HC238, U13 4002, U14 74HC32, U15 74AHC273, U16 CD4532BE, U17 74AHC08, U18 74LS08, U19 74AHC138, U2 74AHC273, U20 74AHC04, U21 74AHC574, U22 74AHC138, U23 4078, U24 74HC11, U25 74LS32, U26 4075, U27 74AHC574, U28 74LS21, U29 74AHC244, U3 74HC74, U30 74AHC02, U31 74AHC138, U32 74HC238, U33 74AHC138, U34 74HC163, U35 74HC238, U36 74LS573, U37 74HC32, U38 74AHC04, U39 74AHC04, U4 74AHC04, U40 74HC00, U41 74HC02, U42 74AHC04, U43 74LS08, U44 74HC32, U45 74AHC273, U46 74AHC273, U47 74AHC04, U49 74AHC244, U5 74AHC08, U50 74AHC244, U51 27C080, U52 74LS08, U53 74HC193, U54 74HC193, U55 74HC157, U56 74AHC273, U57 4078, U58 74AHC244, U59 74HC74, U6 74HC595, U60 74HC283, U61 74HC283, U62 74AHC244, U63 4078, U64 74AHC574, U65 74HC193, U66 74HC193, U67 74HC157, U68 74HC157, U69 74AHC273, U7 74HC165, U70 74HC253, U71 74AHC273, U72 74HC253, U73 74HC253, U74 74AHC273, U75 74LS257, U76 74LS257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

Commit message: Fix KiCad files
Parts:
- added U62, U63: 74HC283, Package_DIP:DIP-16_W7.62mm_Socket_LongPads, symbol 74xx:74LS283
- renumbered U18 to U15, U17 to U16, U15 to U17, U16 to U18, U41 to U28, U37 to U36, U38 to U37, U39 to U38, U40 to U39, U42 to U40, U43 to U41, U44 to U42, U45 to U43, U46 to U44, U47 to U45, U49 to U46, U50 to U47, U51 to U48, U52 to U49, U28 to U50, U53 to U51, U54 to U52, U55 to U53, U56 to U54, U57 to U55, U58 to U56, U59 to U57, U60 to U58, U61 to U59, U62 to U60, U63 to U61, U82 to U64, U64 to U65, U65 to U66, U66 to U67, U67 to U68, U68 to U69, U69 to U70, U70 to U71, U71 to U72, U72 to U73, U73 to U74, U74 to U75, U75 to U76, U76 to U77, U77 to U78, U78 to U79, U79 to U80, U80 to U81, U81 to U82, U90 to U89, U93 to U90, U92 to U91, U36 to U92, U89 to U93
Connections:
- net +5V: now also U90.30 (CS2), U62.16 (VCC), U63.16 (VCC)
- net DB0: now also U63.5 (A1); no longer U69.3 (I1a)
- net DB1: now also U63.3 (A2); no longer U69.6 (I1b)
- net DB2: now also U63.14 (A3); no longer U69.10 (I1c)
- net DB3: now also U63.12 (A4); no longer U69.13 (I1d)
- net DB4: now also U63.6 (B1); no longer U68.3 (I1a)
- net DB5: now also U63.2 (B2); no longer U68.6 (I1b)
- net DB6: now also U63.15 (B3); no longer U68.10 (I1c)
- net DB7: now also U63.11 (B4); no longer U68.13 (I1d)
- net GND: now also U62.7 (C0), U62.8 (GND), U63.8 (GND)
- net O0: now also U62.5 (A1)
- net O1: now also U62.3 (A2)
- net O2: now also U62.14 (A3)
- net O3: now also U62.12 (A4)
- net O4: now also U62.6 (B1)
- net O5: now also U62.2 (B2)
- net O6: now also U62.15 (B3)
- net O7: now also U62.11 (B4)
- net xW_pre: now also U11.13 (Y2); no longer U11.14 (Y1), U40.3
- net DONE: now reaches U16.6, U23.3
- net xF: now reaches U32.11 (Y4)
- net xF: now also U9.10
- net xT: now reaches U32.12 (Y3)
- net xT: now also U9.5
- net xW: now reaches U32.13 (Y2)
- net xW: now also U40.3
- net xJ: now reaches U32.14 (Y1)
- net xJ: now also U13.3
- net NZFLAG_V renamed NZFLAG_I
- net V0 renamed I0
- net V1 renamed I1
- net V2 renamed I2
- net V3 renamed I3
- net V4 renamed I4
- net V5 renamed I5
- net V6 renamed I6
- net V7 renamed I7
- net xF_pre: no longer names the net of U11.11 (Y4)
- net xF_pre: no longer U9.10
- removed net xJ_pre: U11.13 (Y2), U13.3
- net xT_pre: no longer names the net of U11.12 (Y3)
- net xT_pre: no longer U9.5
- net ~{BOV} renamed ~{BOI}
- net ~{COV} renamed ~{COI}
- net ~{GETV} renamed ~{GETI}
- net ~{PUTV} renamed ~{PUTI}
- net ~{Vx} renamed ~{Ix}
- net ~{xV} renamed ~{xI}
- new net: U62.9 (C4), U63.7 (C0)
- new net REL0: U62.4 (S1), U69.3 (I1a)
- new net REL1: U62.1 (S2), U69.6 (I1b)
- new net REL2: U62.13 (S3), U69.10 (I1c)
- new net REL3: U62.10 (S4), U69.13 (I1d)
- new net REL4: U63.4 (S1), U68.3 (I1a)
- new net REL5: U63.1 (S2), U68.6 (I1b)
- new net REL6: U63.13 (S3), U68.10 (I1c)
- new net REL7: U63.10 (S4), U68.13 (I1d)
Other:
- note added: "(Relative jumps)"
- note added: "A/B/R/I SEL"
- note added: "I (INNER Loop Register)"
- note added: "Instruction byte: all0: OPC_SYS 00000 xxx See table @ SYS decoder else: OPC_ADJUST 00001 xxx b2:extended sign bit b1-0 LSB OPC_ALU 0001x xxx See table @ ALU OPC_TRAP 001xx xxx b4:MSB b3-0:LSB (remaining bits set 1) OPC_GETPUT 01xxx xxx b5-4:OFFS b3:GL b2:GP B1-0:ABRV OPC_PAIR 1xxxx xxx DEST SRC"
- note added: "Jump if R not zero"
- note added: "Jump if R zero"
- note added: "Literal Fetch, skip current instruction word Increment PC But NOT if NM"
- note added: "Should implement a "force tristate" pin"
- note added: "W=While Intended to be post decrement"
- note removed: "(Relative addressing here, removed; Just an adder DB+R that feeds into the two 157's on the right instead of their DB input.)"
- note removed: "A/B/R/V SEL"
- note removed: "Bus output use xP, then tristate POR with RDY"
- note removed: "Instruction byte: all0: OPC_SYS 00000 xxx See table @ SYS decoder else: OPC_ADJUST 00001 xxx b2-0 encode signed offset, see table @ R adjust OPC_ALU 0001x xxx See table @ ALU OPC_TRAP 001xx xxx b4:MSB b3-0:LSB (remaining bits set 1) OPC_GETPUT 01xxx xxx b5-4:OFFS b3:GL b2:GP B1-0:ABRV OPC_PAIR 1xxxx xxx DEST SRC"
- note removed: "Jump if xMx not zero"
- note removed: "Jump if xMx zero"
- note removed: "Literal Fetch, skip current instruction word Increment PC immediately"
- note removed: "V (Value Register)"
- note removed: "W=While"
- note removed: "xF"
- note removed: "xJ"
- note removed: "xT"
- note removed: "xW"

Commit message: Add relative JUMPs and add decoders to E register
Parts:
- removed U64: 74AHC04, Package_DIP:DIP-14_W7.62mm_Socket_LongPads, symbol 74xx:74HC04
- added U21, U22: 74HC238, Package_DIP:DIP-16_W7.62mm_Socket_LongPads, symbol 74xx_IEEE:74HC238
- added U27, U28: 74AHC138, Package_DIP:DIP-16_W7.62mm_Socket_LongPads, symbol 74xx:74LS138
- renumbered U22 to U23, U23 to U24, U24 to U25, U25 to U26, U26 to U29, U29 to U30, U30 to U31, U31 to U32, U32 to U33, U33 to U34, U34 to U35, U21 to U36, U35 to U37, U36 to U38, U37 to U39, U39 to U40, U28 to U41, U27 to U42, U46 to U45, U47 to U46, U48 to U47, U45 to U48, U40 to U49, U38 to U50, U49 to U51, U41 to U52, U50 to U53, U51 to U54, U52 to U55, U53 to U56, U54 to U57, U55 to U58, U56 to U59, U58 to U60, U59 to U61, U60 to U62, U61 to U63, U62 to U64, U63 to U65, U42 to U66, U65 to U67, U66 to U68, U67 to U69, U68 to U70, U69 to U71, U70 to U72, U57 to U73, U71 to U74, U72 to U75, U73 to U76, U74 to U77, U75 to U79, U76 to U80, U77 to U81, U78 to U82, U79 to U83, U80 to U84, U81 to U85, U82 to U86, U83 to U87, U84 to U88, U85 to U89, U86 to U90, U87 to U91, U88 to U92, U89 to U93, U90 to U94, U91 to U95, U92 to U96, U93 to U97
Connections:
- net +5V: now also U3.10 (~{S}), U3.13 (~{R}), U21.16 (VCC), U21.6 (G1), U22.16 (VCC), U27.16 (VCC), U27.6 (E3), U28.16 (VCC)
- net DC_pre: now also U50.9
- net DONE: now also U16.3, U20.13; no longer U16.6
- net EH0: now also U21.1 (A0), U22.1 (A0)
- net EH1: now also U21.2 (A1), U22.2 (A1)
- net EH2: now also U21.3 (A2), U22.3 (A2)
- net EH3: now also U21.4 (~{G2A}), U22.6 (G1)
- net EL0: now also U27.1 (A0), U28.1 (A0)
- net EL1: now also U27.2 (A1), U28.2 (A1)
- net EL2: now also U27.3 (A2), U28.3 (A2)
- net EL3: now also U27.4 (E1), U28.6 (E3)
- net GND: now also U41.8, U41.9, U21.5 (~{G2B}), U21.8 (GND), U22.4 (~{G2A}), U22.5 (~{G2B}), U22.8 (GND), U27.5 (E2), U27.8 (GND), U28.4 (E1), U28.5 (E2), U28.8 (GND); no longer U50.5, U50.9
- net GorL: now also U50.5
- net IB3: now also U39.1
- net LO6: now also U49.13
- net RES: no longer U41.8
- net ~{GorL}: now also U50.6
- net ~{Px}: no longer U49.13
- net ~{RET}: now also U23.10 (O5); no longer U23.15 (O0)
- net ~{xP}: no longer U3.13 (~{R})
- net at U41.10: no longer U3.10 (~{S})
- net at U52.5: now also U49.12
- net at U51.2: now also U39.2
- net at U50.8: now also U97.11 (Load)
- removed net NOP: U16.3, U20.13, U24.2
- net Px renamed DH1
- net DH1: now also U21.14 (Y1); no longer U49.12
- removed net RDY: U39.2, U41.9
- net ~{POE}: no longer names the net of U3.9 (Q)
- net ~{POE}: no longer U36.1 (OE)
- removed net ~{RDY}: U23.10 (O5), U39.1
- new net: U16.6, U24.2
- new net DH10: U22.13 (Y2)
- new net DH11: U22.12 (Y3)
- new net DH12: U22.11 (Y4)
- new net DH13: U22.10 (Y5)
- new net DH14: U22.9 (Y6)
- new net DH15: U22.7 (Y7)
- new net DH2: U21.13 (Y2)
- new net DH3: U21.12 (Y3)
- new net DH4: U21.11 (Y4)
- new net DH5: U21.10 (Y5)
- new net DH6: U21.9 (Y6)
- new net DH7: U21.7 (Y7)
- new net DH8: U22.15 (Y0)
- new net DH9: U22.14 (Y1)
- new net ~{DL10}: U28.13 (O2)
- new net ~{DL11}: U28.12 (O3)
- new net ~{DL12}: U28.11 (O4)
- new net ~{DL13}: U28.10 (O5)
- new net ~{DL14}: U28.9 (O6)
- new net ~{DL15}: U28.7 (O7)
- new net ~{DL1}: U27.14 (O1), U36.1 (OE)
- new net ~{DL2}: U27.13 (O2)
- new net ~{DL3}: U27.12 (O3)
- new net ~{DL4}: U27.11 (O4)
- new net ~{DL5}: U27.10 (O5)
- new net ~{DL6}: U27.9 (O6)
- new net ~{DL7}: U27.7 (O7)
- new net ~{DL8}: U28.15 (O0)
- new net ~{DL9}: U28.14 (O1)
- new net ~{NOP}: U23.15 (O0)
- no-connect marks 63 -> 92
Other:
- note added: "ACTIVE HIGH ENABLE"
- note added: "ACTIVE LOW ENABLE"
- note removed: "Should implement a "force tristate" pin"
- moved on the sheet: RN1, RN2, U13C, U14E, U15E, U16B, U16E, U1E, U20G, U25D, U26E, U29A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

Commit message: Add folder structure move files
Connections:
- net DH1 renamed PAR_CP
- net DONE: no longer names the net of U16.3, U20.13, U24.3
- net ~{DL1} renamed ~{PAR_OE}
Other:
- note added: "Currently NOP, reserved for instruction set extension"
- note added: "NULL device"
- note removed: "All NOP, but reserved for instruction set extension except NM"
Changed lines of the file:
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@@
 		(title "Sonne-8 Micro-Controller")
 		(date "2024-08-13")
-		(rev "Myth")
+		(rev "Myth Cut")
 		(company "Contact: mim@ok-schalter.de")
 		(comment 1 "Author: Michael Mangelsdorf")
-		(comment 2 "Project homepage: https://github.com/Dosflange/Sonne")
+		(comment 2 "Project homepage: https://github.com/Dosflange/Myth")
 	)
 	(junction
@@
 		)
 	)
+	(text "NULL device"
+		(exclude_from_sim no)
+		(at 313.568 665.1714 0)
+		(effects
+			(font
+				(size 1.2954 1.2954)
+			)
+			(justify left bottom)
+		)
+	)
 	(text "Device Enable"
 		(exclude_from_sim no)
@@
 		)
 	)
-	(text "All NOP, but\nreserved for\ninstruction set\nextension except NM"
+	(text "Currently NOP,\nreserved for\ninstruction set\nextension"
 		(exclude_from_sim no)
-		(at 221.9927 236.4316 0)
+		(at 216.1811 235.5258 0)
 		(effects
 			(font
@@
 		)
 	)
+	(text "NULL device"
+		(exclude_from_sim no)
+		(at 266.8398 664.8491 0)
+		(effects
+			(font
+				(size 1.2954 1.2954)
+			)
+			(justify left bottom)
+		)
+	)
 	(text "IF GETPUT:\nIB3 set = GLOBAL\nIB3 clear = LOCAL"
 		(exclude_from_sim no)
@@
 		)
 	)
-	(label "DH1"
+	(label "PAR_CP"
 		(at 265.5861 668.8871 0)
 		(fields_autoplaced yes)
@@
 		)
 	)
+	(label "~{PAR_OE}"
+		(at 368.6461 740.792 180)
+		(fields_autoplaced yes)
+		(effects
+			(font
+				(size 1.27 1.27)
+			)
+			(justify right bottom)
+		)
+	)
 	(label "IO1"
 		(at 121.7422 54.5846 180)
@@
 		)
 	)
+	(label "PAR_CP"
+		(at 425.7961 686.182 180)
+		(fields_autoplaced yes)
+		(effects
+			(font
+				(size 1.27 1.27)
+			)
+			(justify right bottom)
+		)
+	)
 	(label "DB7"
 		(at 49.657 360.9848 180)
@@
 		)
 	)
-	(label "DONE"
-		(at 223.3747 279.1714 0)
-		(fields_autoplaced yes)
-		(effects
-			(font
-				(size 1.27 1.27)
-			)
-			(justify left bottom)
-		)
-	)
 	(label "~{GETI}"
 		(at 576.199 717.1182 180)
@@
 		)
 	)
-	(label "DH1"
-		(at 425.7961 686.182 180)
-		(fields_autoplaced yes)
-		(effects
-			(font
-				(size 1.27 1.27)
-			)
-			(justify right bottom)
-		)
-	)
 	(label "~{CLEAR}"
 		(at 821.1312 221.488 180)
@@
 		)
 	)
-	(label "~{DL1}"
-		(at 368.6461 740.792 180)
-		(fields_autoplaced yes)
-		(effects
-			(font
-				(size 1.27 1.27)
-			)
-			(justify right bottom)
-		)
-	)
 	(label "R2"
 		(at 680.0596 421.2844 180)
@@
 		)
 	)
-	(label "~{DL1}"
+	(label "~{PAR_OE}"
 		(at 312.039 669.0831 0)
 		(fields_autoplaced yes)

Commit message: Identify xMx with O
Parts:
- removed U75: 74AHC273, Package_DIP:DIP-20_W7.62mm_Socket_LongPads, symbol 74xx:74HC273
Connections:
- net GND: no longer U13.12
- net O0: now also U80.11 (I0d)
- net O1: now also U80.14 (I0c)
- net O2: now also U80.5 (I0b)
- net O3: now also U80.2 (I0a)
- net O4: now also U81.11 (I0d)
- net O5: now also U81.14 (I0c)
- net O6: now also U81.5 (I0b)
- net O7: now also U81.2 (I0a)
- net at U26.8: now also U13.12
Other:
- note removed: "(Implied address offset for xMx)"
- moved on the sheet: C1, C10, C11, C12, C13, C14, C15, C16, C17, C18, C19, C2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

Commit message: Identify R register and B accumulator
Parts:
- removed U44: 74AHC273, Package_DIP:DIP-20_W7.62mm_Socket_LongPads, symbol 74xx:74HC273
- removed U46: 74AHC244, Package_DIP:DIP-20_W7.62mm_Socket_LongPads, symbol 74xx:74AHC244
- added U52, U73: 74AHC273, Package_DIP:DIP-20_W7.62mm_Socket_LongPads, symbol 74xx:74HC273
- renumbered U42 to U41, U53 to U42, U48 to U43, U49 to U44, U41 to U45, U52 to U46, U56 to U47, U57 to U48, U50 to U49, U60 to U50, U61 to U51, U54 to U53, U55 to U54, U43 to U55, U62 to U56, U67 to U57, U45 to U60, U47 to U61, U63 to U62, U73 to U63, U68 to U67, U69 to U68, U72 to U69, U74 to U72, U51 to U74, U76 to U75, U77 to U76, U79 to U77, U80 to U78, U81 to U79, U82 to U80, U85 to U81, U83 to U82, U84 to U83, U86 to U84, U87 to U85, U88 to U86, U89 to U87, U90 to U88, U91 to U89, U92 to U90, U93 to U91, U94 to U92, U95 to U93, U96 to U94, U97 to U95
Connections:
- net B0 is gone; now on net A0: U55.2 (Q0), U60.2 (1A0), U61.27 (A8)
- net B1 is gone; now on net A1: U55.5 (Q1), U60.4 (1A1), U61.26 (A9)
- net B2 is gone; now on net A2: U55.6 (Q2), U60.6 (1A2), U61.23 (A10)
- net B3 is gone; now on net A3: U55.9 (Q3), U60.8 (1A3), U61.25 (A11)
- net B4 is gone; now on net A4: U55.12 (Q4), U60.17 (2A0), U61.4 (A12)
- net B5 is gone; now on net A5: U55.15 (Q5), U60.15 (2A1), U61.28 (A13)
- net B6 is gone; now on net A6: U55.16 (Q6), U60.13 (2A2), U61.29 (A14)
- net B7 is gone; now on net A7: U55.19 (Q7), U60.11 (2A3), U61.3 (A15)
- net +5V: now also U52.20 (VCC), U73.20 (VCC); no longer U42.13, U89.4 (DOWN), U89.5 (UP)
- net A0: no longer U61.12 (A0)
- net A1: no longer U61.11 (A1)
- net A2: no longer U61.10 (A2)
- net A3: no longer U61.9 (A3)
- net A4: no longer U61.8 (A4)
- net A5: no longer U61.7 (A5)
- net A6: no longer U61.6 (A6)
- net A7: no longer U61.5 (A7)
- net CLOSE: now also U52.11 (Cp), U73.11 (Cp)
- net GND: now also U15.10, U15.9, U26.10, U26.9, U45.2, U45.3, U52.10 (GND), U73.10 (GND)
- net O0: now also U73.3 (D0); no longer U78.11 (I0d)
- net O1: now also U73.4 (D1); no longer U78.14 (I0c)
- net O2: now also U73.7 (D2); no longer U78.5 (I0b)
- net O3: now also U73.8 (D3); no longer U78.2 (I0a)
- net O4: now also U73.13 (D4); no longer U79.11 (I0d)
- net O5: now also U73.14 (D5); no longer U79.14 (I0c)
- net O6: now also U73.17 (D6); no longer U79.5 (I0b)
- net O7: now also U73.18 (D7); no longer U79.2 (I0a)
- net R0: now also U52.3 (D0)
- net R1: now also U52.4 (D1)
- net R2: now also U52.7 (D2)
- net R3: now also U52.8 (D3)
- net R4: now also U52.13 (D4)
- net R5: now also U52.14 (D5)
- net R6: now also U52.17 (D6)
- net R7: now also U52.18 (D7)
- net ~{Dx}: now also U5.10; no longer U5.5
- net ~{GETA}: now also U16.10; no longer U15.9
- net ~{GETR}: now also U8.14 (O1); no longer U8.13 (O2)
- net ~{Ix}: now also U59.1 (1OE), U59.19 (2OE); no longer U5.9
- net ~{Mx}: now also U89.5 (UP)
- net ~{Ox}: now also U74.13; no longer U94.1 (OE)
- net ~{PH3}: no longer U45.2
- net ~{PUTA}: now also U60.1 (1OE), U60.19 (2OE)
- net ~{PUTR}: now also U25.4, U8.10 (O5); no longer U25.11, U8.9 (O6)
- net ~{RES}: now also U52.1 (~{Mr}), U73.1 (~{Mr})
- net ~{xA}: now also U16.9; no longer U15.10
- net ~{xI}: now also U53.11 (~{LOAD}), U54.11 (~{LOAD}); no longer U74.12
- net ~{xM}: now also U89.4 (DOWN)
- net at U15.8: no longer U45.3
- net at U26.8: no longer U13.12
- net into_A: no longer names the net of U45.1
- net into_A: no longer U26.9
- net into_B: no longer names the net of U45.4, U55.11 (Cp)
- net into_B: no longer U26.10
- net xB: no longer names the net of U33.7 (Y7)
- net xB: no longer U44.1
- removed net ~{GETB}: U16.10, U8.14 (O1)
- net ~{GETI} renamed ~{GETD}
- net ~{GETD}: now also U42.13; no longer U74.13
- removed net ~{PUTB}: U25.4, U60.1 (1OE), U60.19 (2OE), U8.10 (O5)
- net ~{PUTI} renamed ~{PUTD}
- net ~{PUTD}: now also U5.9; no longer U5.10
- net ~{xB} renamed GETO
- net GETO: now also U13.12; no longer U16.9
- new net: U5.5, U5.8
- new net: U52.12 (Q4), U61.8 (A4)
- new net: U52.15 (Q5), U61.7 (A5)
- new net: U52.16 (Q6), U61.6 (A6)
- new net: U52.19 (Q7), U61.5 (A7)
- new net: U52.2 (Q0), U61.12 (A0)
- new net: U52.5 (Q1), U61.11 (A1)
- new net: U52.6 (Q2), U61.10 (A2)
- new net: U52.9 (Q3), U61.9 (A3)
- new net: U73.12 (Q4), U78.2 (I0a)
- new net: U73.15 (Q5), U78.5 (I0b)
- new net: U73.16 (Q6), U78.14 (I0c)
- new net: U73.19 (Q7), U78.11 (I0d)
- new net: U73.2 (Q0), U79.2 (I0a)
- new net: U73.5 (Q1), U79.5 (I0b)
- new net: U73.6 (Q2), U79.14 (I0c)
- new net: U73.9 (Q3), U79.11 (I0d)
- new net: U74.11, U94.1 (OE)
- new net ~{GETO}: U44.1, U8.13 (O2)
- new net ~{PUTO}: U25.11, U74.12, U8.9 (O6)
- no-connect marks 92 -> 95
Other:
- note added: "0 IDR ("Identity R" / R:=R) 1 IDA ("Identity A" / R:=A) 2 OCR ("Ones Complement R" / R:=~R) 3 OCA ("Ones Complement A" / R:=~A) 4 SLR ("Shift left R" / R:=R<<1) 5 SLA ("Shift left A" / R:=A<<1) 6 SRR ("Shift right R" / R:=R>>1) 7 SRA ("Shift right A" / R:=A>>1)"
- note added: "8 AND (R:=A&B) 9 IOR (R:=R|A) 10 EOR (R:=R^A) 11 ADD (Add" / R:=R+A, bits 0-7) 12 CAR ("Carry Bit" / R:= Carry, 9th bit of R+A) 00h or 01h 13 RLA ("Flag: R less than A" / R:= (R<A)? 0xEF:0 14 REA ("Flag: R equals A" / R:= (R==A)? 0xEF:0 15 RGA ("Flag: R greater than A" / R:= (R>A)? 0xEF:0"
- note added: "A/R/O/D SEL"
- note added: "Post-inc/dec on DATA RD/WR"
- note added: "R"
- note added: "Zero detection"
- note removed: "0 IDA ("Identity A" / F:=A) 1 IDB ("Identity B" / F:=B) 2 OCA ("Ones Complement A" / F:=~A) 3 OCB ("Ones Complement B" / F:=~B) 4 SLA ("Shift left A" / F:=A<<1) 5 SLB ("Shift left B" / F:=B<<1) 6 SRA ("Shift right A" / F:=A>>1) 7 SRB ("Shift right B" / F:=B>>1)"
- note removed: "8 AND (F:=A&B) 9 IOR (F:=A|B) 10 EOR (F:=A^B) 11 ADD ("Add" / F:=A+B, bits 0-7) 12 CYB ("Carry Bit" / F:= Carry, 9th bit of A+B) 00h or 01h 13 ALB ("Flag: A less than B" / F:= (A<B)? 0xEF:0 14 AEB ("Flag: A equals B" / F:= (A==B)? 0xEF:0 15 AGB ("Flag: A greater than B" / F:= (A>B)? 0xEF:0"
- note removed: "A/B/R/I SEL"
- note removed: "B"
- moved on the sheet: U15C, U16C, U26C, U29B, U3B, U42A, U45A, U45B, U45C, U45D, U47, U48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

Commit message: Change GETPUT, add Q register
Parts:
- removed U5: 74AHC08, Package_DIP:DIP-14_W7.62mm_Socket_LongPads, symbol 74xx:74LS08
- removed U60: 74AHC244, Package_DIP:DIP-20_W7.62mm_Socket_LongPads, symbol 74xx:74AHC244
- removed U8: 74AHC138, Package_DIP:DIP-16_W7.62mm_Socket_LongPads, symbol 74xx:74LS138
- removed U91: 74AHC273, Package_DIP:DIP-20_W7.62mm_Socket_LongPads, symbol 74xx:74HC273
- removed U95: 74LS573, symbol 74xx:74LS573
- added U66: 74AHC273, Package_DIP:DIP-20_W7.62mm_Socket_LongPads, symbol 74xx:74HC273
- added U67: 74AHC244, Package_DIP:DIP-20_W7.62mm_Socket_LongPads, symbol 74xx:74AHC244
- added U9: 74LS139, symbol 74xx:74LS139
- added U92: 74AHC574, Package_DIP:DIP-20_W7.62mm_Socket_LongPads, symbol 74xx:74LS574
- renumbered U17 to U16, U18 to U17, U19 to U18, U20 to U19, U21 to U20, U22 to U21, U23 to U22, U24 to U23, U25 to U24, U26 to U25, U27 to U26, U28 to U27, U29 to U28, U30 to U29, U31 to U30, U32 to U31, U33 to U32, U34 to U33, U35 to U34, U36 to U35, U37 to U36, U38 to U37, U39 to U38, U40 to U39, U41 to U40, U42 to U41, U45 to U42, U47 to U43, U48 to U44, U43 to U45, U44 to U46, U46 to U47, U50 to U48, U51 to U49, U16 to U5, U52 to U50, U55 to U51, U49 to U52, U56 to U55, U57 to U56, U61 to U57, U62 to U58, U58 to U59, U59 to U60, U63 to U61, U69 to U62, U64 to U63, U65 to U64, U66 to U65, U67 to U68, U68 to U69, U9 to U8, U80 to U81, U81 to U82, U82 to U83, U83 to U84, U84 to U85, U85 to U86, U86 to U87, U87 to U88, U88 to U89, U89 to U90, U90 to U91, U92 to U93, U93 to U94, U94 to U95
Connections:
- net ~{GETA} is gone; now on net xW_pre: U5.10
- net ~{GETD} is gone; now on net GND: U41.13
- net ~{PUTA} is gone; now on net ~{PUTR}: U24.5
- net ~{PUTD} is gone; now on net GND: U24.10
- net +5V: now also U66.20 (VCC), U67.20 (VCC), U9.16 (VCC), U92.20 (VCC); no longer U85.6 (1A2)
- net CLOSE: now also U5.12
- net D0: now also U66.2 (Q0), U67.2 (1A0)
- net D1: now also U66.5 (Q1), U67.4 (1A1)
- net D2: now also U66.6 (Q2), U67.6 (1A2)
- net D3: now also U66.9 (Q3), U67.8 (1A3)
- net D4: now also U66.12 (Q4), U67.17 (2A0)
- net D5: now also U66.15 (Q5), U67.15 (2A1)
- net D6: now also U66.16 (Q6), U67.13 (2A2)
- net D7: now also U66.19 (Q7), U67.11 (2A3)
- net DB0: now also U66.3 (D0), U67.18 (1Y0), U92.19 (Q0)
- net DB1: now also U66.4 (D1), U67.16 (1Y1), U92.18 (Q1)
- net DB2: now also U66.7 (D2), U67.14 (1Y2), U92.17 (Q2)
- net DB3: now also U66.8 (D3), U67.12 (1Y3), U92.16 (Q3)
- net DB4: now also U66.13 (D4), U67.3 (2Y0), U92.15 (Q4)
- net DB5: now also U66.14 (D5), U67.5 (2Y1), U92.14 (Q5)
- net DB6: now also U66.17 (D6), U67.7 (2Y2), U92.13 (Q6)
- net DB7: now also U66.18 (D7), U67.9 (2Y3), U92.12 (Q7)
- net GND: now also U24.11, U24.9, U41.10, U41.12, U41.9, U45.9, U52.9, U66.10 (GND), U67.10 (GND), U9.13 (A1), U9.14 (A0), U9.15 (E), U9.8 (GND), U92.10 (GND); no longer U25.10, U25.9, U28.1, U28.2, U28.8, U37.12, U37.13
- net IB0: now also U9.2 (A0)
- net IB1: now also U9.3 (A1)
- net IB2: now also U15.4, U38.1
- net IB3: now also U85.2 (1A0); no longer U15.4, U38.1
- net IB4: now also U85.4 (1A1); no longer U85.2 (1A0)
- net IB5: now also U85.6 (1A2); no longer U85.4 (1A1)
- net NZFLAG_I: now also U5.9
- net TRAP: now also U25.9, U28.1
- net xA: now also U32.14 (Y1); no longer U32.9 (Y6)
- net xC: now also U25.10, U28.2, U32.9 (Y6); no longer U32.10 (Y5), U45.9
- net xC_pre: now also U11.9 (Y6); no longer U11.10 (Y5), U5.13
- net xD: now also U37.12
- net xF: now also U32.10 (Y5); no longer U32.11 (Y4)
- net xJ: now also U32.13 (Y2); no longer U32.14 (Y1)
- net xT: now also U32.11 (Y4); no longer U32.12 (Y3)
- net xW: now also U32.12 (Y3); no longer U32.13 (Y2)
- net xW_pre: now also U11.12 (Y3); no longer U11.13 (Y2)
- net ~{CLEAR}: now also U68.4 (DOWN)
- net ~{Dx}: now also U67.1 (1OE), U67.19 (2OE)
- net ~{GETO}: now also U9.5 (O1)
- net ~{GETPUT}: now also U9.1 (E)
- net ~{GETR}: now also U9.4 (O0)
- net ~{PUTO}: now also U24.4, U9.7 (O3); no longer U24.11
- net ~{PUTR}: now also U9.6 (O2); no longer U24.4
- net ~{RES}: now also U66.1 (~{Mr})
- net ~{RET}: now also U68.5 (UP), U92.1 (OE)
- net ~{TRAP}: no longer U41.9
- net ~{xA}: now also U42.5; no longer U5.9
- net ~{xD}: no longer U41.12
- net ~{xM}: now also U24.3; no longer U24.9
- net at U37.1: now also U5.11
- net at U61.9 (Q): now also U5.13
- net at U37.11: now also U66.11 (Cp)
- net at U5.8: now also U13.2; no longer U42.5
- net at U28.9: now also U92.11 (Cp)
- net at U89.12 (Zd): now also U92.9 (D7)
- net at U89.4 (Za): now also U92.6 (D4)
- net at U89.7 (Zb): now also U92.7 (D5)
- net at U89.9 (Zc): now also U92.8 (D6)
- net xQ: now reaches U32.7 (Y7)
- net xQ: now also U28.8
- net at U88.4 (Za): now also U92.2 (D0)
- net at U88.7 (Zb): now also U92.3 (D1)
- net at U88.9 (Zc): now also U92.4 (D2)
- net at U88.12 (Zd): now also U92.5 (D3)
- net at U25.8: now also U37.13
- net at U24.8: no longer U24.3
- net A0: no longer names the net of U51.2 (Q0), U57.27 (A8)
- net A1: no longer names the net of U51.5 (Q1), U57.26 (A9)
- net A2: no longer names the net of U51.6 (Q2), U57.23 (A10)
- net A3: no longer names the net of U51.9 (Q3), U57.25 (A11)
- net A4: no longer names the net of U51.12 (Q4), U57.4 (A12)
- net A5: no longer names the net of U51.15 (Q5), U57.28 (A13)
- net A6: no longer names the net of U51.16 (Q6), U57.29 (A14)
- net A7: no longer names the net of U51.19 (Q7), U57.3 (A15)
- removed net DC_pre: U5.11, U52.9
- net Dx_pre: no longer names the net of U12.13 (Y2)
- net Dx_pre: no longer U5.12
- net ~{NEW}: no longer names the net of U22.9 (O6)
- net ~{NEW}: no longer U68.4 (DOWN)
- net ~{OLD}: no longer names the net of U22.7 (O7)
- net ~{OLD}: no longer U68.5 (UP)
- net ~{xC}: no longer names the net of U45.8
- net ~{xC}: no longer U41.10
- no-connect marks 95 -> 103
Other:
- note added: "(DATA) Segment index"
- note added: "(GLOBAL) Segment index"
- note added: "(QUIT) page index Stored return page during calls"
- note added: "8 AND (R:=R&A) 9 IOR (R:=R|A) 10 EOR (R:=R^A) 11 ADD (Add" / R:=R+A, bits 0-7) 12 CAR ("Carry Bit" / R:= Carry, 9th bit of R+A) 00h or 01h 13 RLA ("Flag: R less than A" / R:= (R<A)? 0xFF:0 14 REA ("Flag: R equals A" / R:= (R==A)? 0xFF:0 15 RGA ("Flag: R greater than A" / R:= (R>A)? 0xFF:0"
- note added: "Automatic call stack CALL: Enter stack frame RET: Resume previous frame"
- note added: "G"
- note added: "IB 3-5 are the immediate offset for GET-PUT operations"
- note added: "IB2 is global/local IB3-5 is byte offset"
- note added: "IF GETPUT: IB2 set = GLOBAL IB2 clear = LOCAL"
- note added: "Instruction byte: all0: OPC_SYS 00000 xxx See table @ SYS decoder else: OPC_ADJUST 00001 xxx b2:extended sign bit b1-0 LSB OPC_ALU 0001x xxx See table @ ALU OPC_TRAP 001xx xxx b4:MSB b3-0:LSB (remaining bits set 1) OPC_GETPUT 01xxx xxx b5-3 OFFS b2:GL b1:GP B0:RO OPC_PAIR 1xxxx xxx DEST SRC"
- note added: "L (LOCAL) Segment index (Stack Pointer)"
- note added: "Myth Microcontroller Reference Schematics"
- note added: "Q"
- note added: "R/O"
- note removed: "8 AND (R:=A&B) 9 IOR (R:=R|A) 10 EOR (R:=R^A) 11 ADD (Add" / R:=R+A, bits 0-7) 12 CAR ("Carry Bit" / R:= Carry, 9th bit of R+A) 00h or 01h 13 RLA ("Flag: R less than A" / R:= (R<A)? 0xEF:0 14 REA ("Flag: R equals A" / R:= (R==A)? 0xEF:0 15 RGA ("Flag: R greater than A" / R:= (R>A)? 0xEF:0"
- note removed: "A/R/O/D SEL"
- note removed: "D(ata) page index"
- note removed: "IB 4,5 are the hardcoded offset for GET-PUT operations"
- note removed: "IB3 is global/local"
- note removed: "IF GETPUT: IB3 set = GLOBAL IB3 clear = LOCAL"
- note removed: "Instruction byte: all0: OPC_SYS 00000 xxx See table @ SYS decoder else: OPC_ADJUST 00001 xxx b2:extended sign bit b1-0 LSB OPC_ALU 0001x xxx See table @ ALU OPC_TRAP 001xx xxx b4:MSB b3-0:LSB (remaining bits set 1) OPC_GETPUT 01xxx xxx b5-4:OFFS b3:GL b2:GP B1-0:ABRV OPC_PAIR 1xxxx xxx DEST SRC"
- note removed: "L"
- note removed: "L(ocal) page index Stack Pointer"
- note removed: "OLD/NEW create/remove stack frames"
- note removed: "Sonne Microcontroller Reference Schematics rev. Myth"
- moved on the sheet: U15C, U1A, U24C, U25C, U28A, U28B, U30D, U37D, U39A, U39C, U3B, U41A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
