File: Work_in_progress/tools/Schematics/myth.kicad_sch (KiCad schematic)
At the start: 132 parts, among them J1 Conn_01x08_Male, J2 Conn_01x08_Male, J3 Conn_01x08_Male, J4 Conn_01x08_Male, J5 Conn_01x04_Male, J6 Conn_01x04_Male, J7 Conn_02x01, U1 74AHC02, U10 74HC238, U11 74HC238, U12 74HC238, U13 4002, U14 74HC32, U15 74LS08, U16 74AHC273, U17 CD4532BE, U18 74AHC138, U19 74AHC04, U2 74AHC273, U20 74HC238, U21 74HC238, U22 74AHC138, U23 4078, U24 74HC11, U25 74LS32, U26 74AHC138, U27 74AHC138, U28 4075, U29 74AHC244, U3 74HC74, U30 74AHC02, U31 74AHC138, U32 74HC238, U33 74AHC138, U34 74HC163, U35 74AHC574, U36 74HC238, U37 74HC32, U38 74AHC04, U39 74HC00, U4 74AHC04, U40 74AHC574, U41 74LS21, U42 74HC02, U43 74HC157, U44 74AHC273, U45 74AHC04, U46 74AHC04, U47 74LS08, U48 74HC283, U49 74HC283, U5 74AHC08, U50 74AHC273, U51 74AHC273, U52 74AHC04, U53 74HC193, U54 74HC193, U55 74AHC244, U56 74AHC574, U57 27C080, U58 4078, U59 4078, U6 74HC595, U60 74AHC244, U61 74HC74, U62 74AHC273, U63 74HC283, U64 74HC283, U65 74HC32, U66 74AHC273, U67 74AHC244, U68 74HC193, U69 74HC193, U7 74HC165, U70 74HC157, U71 74HC157, U72 74HC253, U73 74AHC273, U74 74LS08, U75 74HC253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

Commit message: Add CALLER to SYS group
Connections:
- net GND: now also U25.10, U25.9; no longer U15.10, U15.9, U39.10, U39.9
- net TRAP: no longer U25.9
- net xC: no longer U25.10
- net xD: no longer U37.12
- net ~{RET}: now also U15.9; no longer U92.1 (OE)
- net ~{xD}: now also U39.9
- net at U37.11: no longer U66.11 (Cp)
- net at U37.13: no longer U25.8
- net ~{CALLER}: now reaches U22.9 (O6)
- net ~{CALLER}: now also U15.10, U39.10
- net at U39.8: now also U66.11 (Cp)
- net at U15.8: now also U92.1 (OE)
Other:
- moved on the sheet: U15C, U25C, U37D, U39C
Changed lines of the file:
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@@
 	)
 	(no_connect
+		(at 879.4455 779.4137)
+	)
+	(no_connect
 		(at 312.1801 720.7427)
 	)
@@
 	)
 	(no_connect
-		(at 273.7866 390.1948)
-	)
-	(no_connect
 		(at 1011.8406 792.8751)
 	)
@@
 	(wire
 		(pts
+			(xy 864.2055 776.8737) (xy 864.2055 781.9537)
+		)
+		(stroke
+			(width 0)
+			(type default)
+		)
+	)
+	(wire
+		(pts
 			(xy 604.2926 383.2313) (xy 604.2926 421.5708)
 		)
@@
 	(wire
 		(pts
+			(xy 1055.7366 657.1742) (xy 1056.9448 657.1742)
+		)
+		(stroke
+			(width 0)
+			(type default)
+		)
+	)
+	(wire
+		(pts
 			(xy 184.658 466.0138) (xy 165.4048 466.0138)
 		)
@@
 	(wire
 		(pts
+			(xy 1055.7366 676.2312) (xy 1055.7366 657.1742)
+		)
+		(stroke
+			(width 0)
+			(type default)
+		)
+	)
+	(wire
+		(pts
 			(xy 785.5784 817.9799) (xy 825.2278 817.9799)
 		)
@@
 	(text "Q"
 		(exclude_from_sim no)
-		(at 1047.9427 698.8803 0)
+		(at 1077.4927 684.8182 0)
 		(effects
 			(font
@@
 		)
 	)
-	(label "TRAP"
-		(at 704.5218 438.9412 180)
-		(fields_autoplaced yes)
-		(effects
-			(font
-				(size 1.27 1.27)
-			)
-			(justify right bottom)
-		)
-	)
 	(label "EH0"
 		(at 237.9045 719.1964 180)
@@
 		)
 	)
-	(label "xD"
+	(label "~{xD}"
 		(at 719.7618 436.4012 180)
 		(fields_autoplaced yes)
@@
 		)
 	)
+	(label "GND"
+		(at 864.2055 776.8737 180)
+		(fields_autoplaced yes)
+		(effects
+			(font
+				(size 1.27 1.27)
+			)
+			(justify right bottom)
+		)
+	)
 	(label "IPH"
 		(at 1072.8452 504.2662 180)
@@
 		)
 	)
+	(label "~{CALLER}"
+		(at 719.7618 441.4812 180)
+		(fields_autoplaced yes)
+		(effects
+			(font
+				(size 1.27 1.27)
+			)
+			(justify right bottom)
+		)
+	)
 	(label "EH1"
 		(at 237.6461 682.8571 180)
@@
 	)
 	(label "~{RET}"
-		(at 1056.9448 657.1742 180)
+		(at 1040.4966 673.6912 180)
 		(fields_autoplaced yes)
 		(effects
@@
 		)
 	)
+	(label "~{CALLER}"
+		(at 273.7866 390.1948 0)
+		(fields_autoplaced yes)
+		(effects
+			(font
+				(size 1.27 1.27)
+			)
+			(justify left bottom)
+		)
+	)
 	(label "GND"
 		(at 897.1276 774.355 180)
@@
 		)
 	)
-	(label "xC"
-		(at 704.5218 444.0212 180)
-		(fields_autoplaced yes)
-		(effects
-			(font
-				(size 1.27 1.27)
-			)
-			(justify right bottom)
-		)
-	)
 	(label "+5V"
 		(at 1075.9948 624.1542 0)
@@
 		)
 	)
+	(label "~{CALLER}"
+		(at 1040.4966 678.7712 180)
+		(fields_autoplaced yes)
+		(effects
+			(font
+				(size 1.27 1.27)
+			)
+			(justify right bottom)
+		)
+	)
 	(label "+5V"
 		(at 911.4282 346.9132 180)
@@
 	(symbol
 		(lib_id "74xx:74LS32")
-		(at 727.3818 438.9412 0)
+		(at 853.3955 769.5629 0)
 		(unit 4)
 		(exclude_from_sim no)
@@
 		(dnp no)
 		(property "Reference" "U37"
-			(at 727.3818 430.6862 0)
+			(at 853.3955 761.3079 0)
 			(effects
 				(font
@@
 		)
 		(property "Value" "74HC32"
-			(at 727.3818 432.9976 0)
+			(at 853.3955 763.6193 0)
 			(effects
 				(font
@@
 		)
 		(property "Footprint" "Package_DIP:DIP-14_W7.62mm_Socket_LongPads"
-			(at 727.3818 438.9412 0)
+			(at 853.3955 769.5629 0)
 			(effects
 				(font
@@
 		)
 		(property "Datasheet" "http://www.ti.com/lit/gpn/sn74LS32"
-			(at 727.3818 438.9412 0)
+			(at 853.3955 769.5629 0)
 			(effects
 				(font
@@
 		)
 		(property "Description" ""
-			(at 727.3818 438.9412 0)
+			(at 853.3955 769.5629 0)
 			(effects
 				(font
@@
 	(symbol
 		(lib_id "74xx:74HC00")
-		(at 905.3058 791.0728 0)
+		(at 727.3818 438.9412 0)
 		(unit 3)
 		(exclude_from_sim no)
@@
 		(fields_autoplaced yes)
 		(property "Reference" "U39"
-			(at 905.2975 783.6828 0)
+			(at 727.3735 431.5512 0)
 			(effects
 				(font
@@
 		)
 		(property "Value" "74HC00"
-			(at 905.2975 785.7308 0)
+			(at 727.3735 433.5992 0)
 			(effects
 				(font
@@
 		)
 		(property "Footprint" "Package_DIP:DIP-14_W7.62mm_Socket_LongPads"
-			(at 905.3058 791.0728 0)
+			(at 727.3818 438.9412 0)
 			(effects
 				(font
@@
 		)
 		(property "Datasheet" "http://www.ti.com/lit/gpn/sn74hc00"
-			(at 905.3058 791.0728 0)
+			(at 727.3818 438.9412 0)
 			(effects
 				(font
@@
 		)
 		(property "Description" ""
-			(at 905.3058 791.0728 0)
+			(at 727.3818 438.9412 0)
 			(effects
 				(font
@@
 	(symbol
 		(lib_id "74xx:74LS32")
-		(at 712.1418 441.4812 0)
+		(at 871.8255 779.4137 0)
 		(unit 3)
 		(exclude_from_sim no)
@@
 		(fields_autoplaced yes)
 		(property "Reference" "U25"
-			(at 712.1418 433.5269 0)
+			(at 871.8255 771.4594 0)
 			(effects
 				(font
@@
 		)
 		(property "Value" "74LS32"
-			(at 712.1418 435.9511 0)
+			(at 871.8255 773.8836 0)
 			(effects
 				(font
@@
 		)
 		(property "Footprint" "Package_DIP:DIP-14_W7.62mm_Socket_LongPads"
-			(at 712.1418 441.4812 0)
+			(at 871.8255 779.4137 0)
 			(effects
 				(font
@@
 		)
 		(property "Datasheet" "http://www.ti.com/lit/gpn/sn74LS32"
-			(at 712.1418 441.4812 0)
+			(at 871.8255 779.4137 0)
 			(effects
 				(font
@@
 		)
 		(property "Description" ""
-			(at 712.1418 441.4812 0)
+			(at 871.8255 779.4137 0)
 			(effects
 				(font
@@
 	(symbol
 		(lib_id "74xx:74LS08")
-		(at 939.8178 778.1147 0)
+		(at 1048.1166 676.2312 0)
 		(unit 3)
 		(exclude_from_sim no)
@@
 		(fields_autoplaced yes)
 		(property "Reference" "U15"
-			(at 939.8095 770.1604 0)
+			(at 1048.1083 668.2769 0)
 			(effects
 				(font
@@
 		)
 		(property "Value" "74LS08"
-			(at 939.8095 772.5846 0)
+			(at 1048.1083 670.7011 0)
 			(effects
 				(font
@@
 		)
 		(property "Footprint" "Package_DIP:DIP-14_W7.62mm_Socket_LongPads"
-			(at 939.8178 778.1147 0)
+			(at 1048.1166 676.2312 0)
 			(effects
 				(font
@@
 		)
 		(property "Datasheet" "http://www.ti.com/lit/gpn/sn74LS08"
-			(at 939.8178 778.1147 0)
+			(at 1048.1166 676.2312 0)
 			(effects
 				(font
@@
 		)
 		(property "Description" ""
-			(at 939.8178 778.1147 0)
+			(at 1048.1166 676.2312 0)
 			(effects
 				(font

Commit message: Revert Q reg to D
Parts:
- removed U67: 74AHC244, Package_DIP:DIP-20_W7.62mm_Socket_LongPads, symbol 74xx:74AHC244
Connections:
- net D0: now also U92.2 (D0)
- net D1: now also U92.3 (D1)
- net D2: now also U92.4 (D2)
- net D3: now also U92.5 (D3)
- net D4: now also U92.6 (D4)
- net D5: now also U92.7 (D5)
- net D6: now also U92.8 (D6)
- net D7: now also U92.9 (D7)
- net DB0: no longer U66.3 (D0)
- net DB1: no longer U66.4 (D1)
- net DB2: no longer U66.7 (D2)
- net DB3: no longer U66.8 (D3)
- net DB4: no longer U66.13 (D4)
- net DB5: no longer U66.14 (D5)
- net DB6: no longer U66.17 (D6)
- net DB7: no longer U66.18 (D7)
- net GND: now also U37.12, U37.13, U39.10, U39.9; no longer U30.11, U30.12, U45.9, U52.9
- net RET: now also U30.11
- net xC_pre: now also U15.10
- net xD: now also U28.8
- net ~{Dx}: now also U52.9
- net ~{RET}: no longer U15.9
- net ~{xD}: no longer U39.9
- net at U45.8: now also U92.11 (Cp)
- net at U28.9: now also U66.11 (Cp); no longer U92.11 (Cp)
- net at U89.12 (Zd): now also U66.18 (D7); no longer U92.9 (D7)
- net at U89.4 (Za): now also U66.13 (D4); no longer U92.6 (D4)
- net at U89.7 (Zb): now also U66.14 (D5); no longer U92.7 (D5)
- net at U89.9 (Zc): now also U66.17 (D6); no longer U92.8 (D6)
- net at U30.13: now also U92.1 (OE)
- net at U39.8: no longer U66.11 (Cp)
- net Dx: now reaches U52.8
- net Dx: now also U30.12
- net at U88.12 (Zd): now also U66.8 (D3); no longer U92.5 (D3)
- net at U88.4 (Za): now also U66.3 (D0); no longer U92.2 (D0)
- net at U88.7 (Zb): now also U66.4 (D1); no longer U92.3 (D1)
- net at U88.9 (Zc): now also U66.7 (D2); no longer U92.4 (D2)
- net Dx_pre: now reaches U12.13 (Y2)
- net Dx_pre: now also U15.9
- net DC_pre: now reaches U15.8
- net DC_pre: now also U45.9; no longer U92.1 (OE)
- net xQ: no longer names the net of U32.7 (Y7)
- net xQ: no longer U28.8
- removed net ~{CALLER}: U15.10, U22.9 (O6), U39.10
- no-connect marks 103 -> 101
Other:
- note removed: "(QUIT) page index Stored return page during calls"
- note removed: "Q"
- moved on the sheet: U15C, U25C, U30D, U37D, U39C, U45D, U52D, U62, U66, U92
