File: Work_in_progress/tools/Schematics/myth.kicad_sch (KiCad schematic)
At the start: 131 parts, among them J1 Conn_01x08_Male, J2 Conn_01x08_Male, J3 Conn_01x08_Male, J4 Conn_01x08_Male, J5 Conn_01x04_Male, J6 Conn_01x04_Male, J7 Conn_02x01, U1 74AHC02, U10 74HC238, U11 74HC238, U12 74HC238, U13 4002, U14 74HC32, U15 74LS08, U16 74AHC273, U17 CD4532BE, U18 74AHC138, U19 74AHC04, U2 74AHC273, U20 74HC238, U21 74HC238, U22 74AHC138, U23 4078, U24 74HC11, U25 74LS32, U26 74AHC138, U27 74AHC138, U28 4075, U29 74AHC244, U3 74HC74, U30 74AHC02, U31 74AHC138, U32 74HC238, U33 74AHC138, U34 74HC163, U35 74AHC574, U36 74HC238, U37 74HC32, U38 74AHC04, U39 74HC00, U4 74AHC04, U40 74AHC574, U41 74LS21, U42 74HC02, U43 74HC157, U44 74AHC273, U45 74AHC04, U46 74AHC04, U47 74LS08, U48 74HC283, U49 74HC283, U5 74AHC08, U50 74AHC273, U51 74AHC273, U52 74AHC04, U53 74HC193, U54 74HC193, U55 74AHC244, U56 74AHC574, U57 27C080, U58 4078, U59 4078, U6 74HC595, U60 74AHC244, U61 74HC74, U62 74AHC273, U63 74HC283, U64 74HC283, U65 74HC32, U66 74AHC273, U68 74HC193, U69 74HC193, U7 74HC165, U70 74HC157, U71 74HC157, U72 74HC253, U73 74AHC273, U74 74LS08, U75 74HC253, U76 74HC253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

Commit message: Remove A, try R new/old
Parts:
- added U67: 74AHC273, Package_DIP:DIP-20_W7.62mm_Socket_LongPads, symbol 74xx:74HC273
Connections:
- net +5V: now also U67.20 (VCC)
- net CLOSE: now also U67.11 (Cp)
- net DB0: no longer U51.3 (D0)
- net DB1: no longer U51.4 (D1)
- net DB2: no longer U51.7 (D2)
- net DB3: no longer U51.8 (D3)
- net DB4: no longer U51.13 (D4)
- net DB5: no longer U51.14 (D5)
- net DB6: no longer U51.17 (D6)
- net DB7: no longer U51.18 (D7)
- net GND: now also U42.5, U42.6, U67.10 (GND); no longer U4.3
- net R0: now also U51.3 (D0)
- net R1: now also U51.4 (D1)
- net R2: now also U51.7 (D2)
- net R3: now also U51.8 (D3)
- net R4: now also U51.13 (D4)
- net R5: now also U51.14 (D5)
- net R6: now also U51.17 (D6)
- net R7: now also U51.18 (D7)
- net ~{PH3}: no longer U42.6
- net ~{RES}: now also U67.1 (~{Mr})
- net ~{opc_ALU}: now also U4.3
- net ~{xA}: no longer U42.5
- net opc_ALU: now reaches U4.4
- net opc_ALU: now also U51.11 (Cp)
- net ~{xW}: now reaches U46.4, U53.4 (DOWN)
- net at U42.4: no longer U51.11 (Cp)
- net at U51.12 (Q4): now also U67.13 (D4); no longer U57.4 (A12)
- net at U51.15 (Q5): now also U67.14 (D5); no longer U57.28 (A13)
- net at U51.16 (Q6): now also U67.17 (D6); no longer U57.29 (A14)
- net at U51.19 (Q7): now also U67.18 (D7); no longer U57.3 (A15)
- net at U51.2 (Q0): now also U67.3 (D0); no longer U57.27 (A8)
- net at U51.5 (Q1): now also U67.4 (D1); no longer U57.26 (A9)
- net at U51.6 (Q2): now also U67.7 (D2); no longer U57.23 (A10)
- net at U51.9 (Q3): now also U67.8 (D3); no longer U57.25 (A11)
- new net: U57.23 (A10), U67.6 (Q2)
- new net: U57.25 (A11), U67.9 (Q3)
- new net: U57.26 (A9), U67.5 (Q1)
- new net: U57.27 (A8), U67.2 (Q0)
- new net: U57.28 (A13), U67.15 (Q5)
- new net: U57.29 (A14), U67.16 (Q6)
- new net: U57.3 (A15), U67.19 (Q7)
- new net: U57.4 (A12), U67.12 (Q4)
Other:
- note added: "0 IDN ("Identity New" / New:=New) 1 IDO ("Identity Old" / New:=Old) 2 OCR ("Ones Complement New" / New:=~New) 3 OCA ("Ones Complement Old" / New:=~Old) 4 SLR ("Shift left New" / New:=New<<1) 5 SLA ("Shift left Old" / New:=Old<<1) 6 SRR ("Shift right New" / New:=New>>1) 7 SRA ("Shift right Old" / New:=Old>>1)"
- note added: "8 AND (New:=New&Old) 9 IOR (New:=New|Old) 10 EOR (New:=New^Old) 11 ADD (Add" / New:=New+Old, bits 0-7) 12 CAR ("Carry Bit" / New:= Carry, 9th bit of New+Old) 00h or 01h 13 NLO ("Flag: New less than Old" / New:= (New<Old)? 0xFF:0 14 NEO ("Flag: New equals Old" / New:= (New==Old)? 0xFF:0 15 NGO ("Flag: New greater than Old" / New:= (New>Old)? 0xFF:0"
- note added: "BLUR3 LUT ROM"
- note added: "R new"
- note added: "R old"
- note removed: "0 IDR ("Identity R" / R:=R) 1 IDA ("Identity A" / R:=A) 2 OCR ("Ones Complement R" / R:=~R) 3 OCA ("Ones Complement A" / R:=~A) 4 SLR ("Shift left R" / R:=R<<1) 5 SLA ("Shift left A" / R:=A<<1) 6 SRR ("Shift right R" / R:=R>>1) 7 SRA ("Shift right A" / R:=A>>1)"
- note removed: "8 AND (R:=R&A) 9 IOR (R:=R|A) 10 EOR (R:=R^A) 11 ADD (Add" / R:=R+A, bits 0-7) 12 CAR ("Carry Bit" / R:= Carry, 9th bit of R+A) 00h or 01h 13 RLA ("Flag: R less than A" / R:= (R<A)? 0xFF:0 14 REA ("Flag: R equals A" / R:= (R==A)? 0xFF:0 15 RGA ("Flag: R greater than A" / R:= (R>A)? 0xFF:0"
- note removed: "A"
- note removed: "R"
- moved on the sheet: U42B, U46B, U4B, U51

Commit message: Rework everything
Parts:
- removed unit 3 of U24
- removed unit 3 of U25
- removed U51, U62: 74AHC273, Package_DIP:DIP-20_W7.62mm_Socket_LongPads, symbol 74xx:74HC273
- removed U68, U69, U90, U91: 74HC193, Package_DIP:DIP-16_W7.62mm_Socket_LongPads, symbol 74xx:74LS193
- removed U72, U75, U76, U81: 74HC253, Package_DIP:DIP-16_W7.62mm_Socket_LongPads, symbol 74xx:74LS253
- removed U86, U87: 74HC157, Package_DIP:DIP-16_W7.62mm_Socket_LongPads, symbol 74xx:74LS157
- removed U93: 628128_DIP32_SSOP32, symbol Memory_RAM:628128_DIP32_SSOP32
- removed U95: 74LS573, symbol 74xx:74LS573
- added U51, U62, U68, U72: 74AHC244, Package_DIP:DIP-20_W7.62mm_Socket_LongPads, symbol 74xx:74AHC244
- added U69: 628128_DIP32_SSOP32, symbol Memory_RAM:628128_DIP32_SSOP32
- added U75, U76: 74HC157, Package_DIP:DIP-16_W7.62mm_Socket_LongPads, symbol 74xx:74LS157
- added U81: 74AHC273, Package_DIP:DIP-20_W7.62mm_Socket_LongPads, symbol 74xx:74HC273
- added U98, U99: 74HC193, Package_DIP:DIP-16_W7.62mm_Socket_LongPads, symbol 74xx:74LS193
Connections:
- net D0 is gone; now on net G0: U66.2 (Q0), U92.2 (D0)
- net D1 is gone; now on net G1: U66.5 (Q1), U92.3 (D1)
- net D2 is gone; now on net G2: U66.6 (Q2), U92.4 (D2)
- net D3 is gone; now on net G3: U66.9 (Q3), U92.5 (D3)
- net D4 is gone; now on net G4: U66.12 (Q4), U92.6 (D4)
- net D5 is gone; now on net G5: U66.15 (Q5), U92.7 (D5)
- net D6 is gone; now on net G6: U66.16 (Q6), U92.8 (D6)
- net D7 is gone; now on net G7: U66.19 (Q7), U92.9 (D7)
- net +5V: now also U51.20 (VCC), U62.20 (VCC), U68.20 (VCC), U72.20 (VCC), U75.16 (VCC), U76.16 (VCC), U81.20 (VCC), U98.1 (B), U98.10 (C), U98.11 (~{LOAD}), U98.15 (A), U98.16 (VCC), U98.9 (D), U99.1 (B), U99.10 (C), U99.11 (~{LOAD}), U99.15 (A), U99.16 (VCC), U99.9 (D)
- net C0: now also U72.2 (1A0)
- net C1: now also U72.4 (1A1)
- net C2: now also U72.6 (1A2)
- net C3: now also U72.8 (1A3)
- net C4: now also U72.17 (2A0)
- net C5: now also U72.15 (2A1)
- net C6: now also U72.13 (2A2)
- net C7: now also U72.11 (2A3)
- net DB0: now also U51.18 (1Y0), U69.13 (Q0), U76.3 (I1a)
- net DB1: now also U51.16 (1Y1), U69.14 (Q1), U76.6 (I1b)
- net DB2: now also U51.14 (1Y2), U69.15 (Q2), U76.10 (I1c)
- net DB3: now also U51.12 (1Y3), U69.17 (Q3), U76.13 (I1d)
- net DB4: now also U51.3 (2Y0), U69.18 (Q4), U75.3 (I1a)
- net DB5: now also U51.5 (2Y1), U69.19 (Q5), U75.6 (I1b)
- net DB6: now also U51.7 (2Y2), U69.20 (Q6), U75.10 (I1c)
- net DB7: now also U51.9 (2Y3), U69.21 (Q7), U75.13 (I1d)
- net DC_pre: no longer U45.9
- net Dx: no longer U30.12
- net Dx_pre: no longer U12.13 (Y2)
- net FETCH: now also U1.9; no longer U14.1, U65.1
- net G0: now also U68.2 (1A0)
- net G1: now also U68.4 (1A1)
- net G2: now also U68.6 (1A2)
- net G3: now also U68.8 (1A3)
- net G4: now also U68.17 (2A0)
- net G5: now also U68.15 (2A1)
- net G6: now also U68.13 (2A2)
- net G7: now also U68.11 (2A3)
- net GETO: now also U37.13; no longer U13.12
- net GLOBAL: now also U65.13; no longer U65.10, U65.2
- net GND: now also U51.10 (GND), U62.10 (GND), U68.10 (GND), U72.10 (GND), U75.15 (E), U75.8 (GND), U76.15 (E), U76.8 (GND), U81.10 (GND), U98.8 (GND), U99.8 (GND); no longer U37.12, U37.13, U42.5, U42.6, U42.8, U42.9, U94.29 (A14), U94.3 (A15)
- net GorL: now also U65.11; no longer U47.9, U52.5, U65.5, U65.8, U74.10
- net IB2: no longer U30.9, U38.1
- net J0: now also U76.2 (I0a)
- net J1: now also U76.5 (I0b)
- net J2: now also U76.11 (I0c)
- net J3: now also U76.14 (I0d)
- net J4: now also U75.2 (I0a)
- net J5: now also U75.5 (I0b)
- net J6: now also U75.11 (I0c)
- net J7: now also U75.14 (I0d)
- net JIN0: now also U63.5 (A1)
- net JIN1: now also U63.3 (A2)
- net JIN2: now also U63.14 (A3)
- net JIN3: now also U63.12 (A4)
- net JIN4: now also U63.6 (B1)
- net JIN5: now also U63.2 (B2)
- net JIN6: now also U63.15 (B3)
- net JIN7: now also U63.11 (B4)
- net LO6: now also U94.6 (A6), U69.6 (A6); no longer U47.12
- net LO7: now also U94.5 (A7), U69.5 (A7)
- net LOCAL: now also U65.12; no longer U47.10, U65.9
- net Mx_pre: no longer U12.14 (Y1)
- net Nx_pre: no longer U12.15 (Y0)
- net O0: now also U67.3 (D0), U51.2 (1A0), U81.2 (Q0); no longer U63.5 (A1)
- net O1: now also U67.4 (D1), U51.4 (1A1), U81.5 (Q1); no longer U63.3 (A2)
- net O2: now also U67.7 (D2), U51.6 (1A2), U81.6 (Q2); no longer U63.14 (A3)
- net O3: now also U67.8 (D3), U51.8 (1A3), U81.9 (Q3); no longer U63.12 (A4)
- net O4: now also U67.13 (D4), U51.17 (2A0), U81.12 (Q4); no longer U63.6 (B1)
- net O5: now also U67.14 (D5), U51.15 (2A1), U81.15 (Q5); no longer U63.2 (B2)
- net O6: now also U67.17 (D6), U51.13 (2A2), U81.16 (Q6); no longer U63.15 (B3)
- net O7: now also U67.18 (D7), U51.11 (2A3), U81.19 (Q7); no longer U63.11 (B4)
- net OC_pre: no longer U52.3
- net RES: now also U98.14 (CLR), U99.14 (CLR)
- net TRAP: no longer U13.9
- net xA: no longer U32.14 (Y1)
- net xC: now also U32.7 (Y7), U65.5; no longer U13.10, U32.9 (Y6)
- net xD: no longer U28.8, U88.1 (S), U89.1 (S)
- net xF: now also U32.9 (Y6); no longer U32.10 (Y5)
- net xG: now also U28.8, U88.1 (S), U89.1 (S)
- net xJ: now also U32.12 (Y3); no longer U32.13 (Y2)
- net xM_pre: no longer U10.14 (Y1)
- net xO: now also U37.12; no longer U13.11
- net xT: now also U32.10 (Y5); no longer U32.11 (Y4)
- net xW: now also U32.11 (Y4); no longer U32.12 (Y3)
- net ~{BOL}: now also U98.13 (~{BO}), U99.4 (DOWN)
- net ~{CLEAR}: now also U98.4 (DOWN)
- net ~{COL}: now also U98.12 (~{CO}), U99.5 (UP)
- net ~{Dx}: no longer U31.13 (O2)
- net ~{GETPUT}: no longer U30.8
- net ~{IN_RAM}: now also U69.22 (~{CS1}), U69.30 (CS2)
- net ~{IN_ROM}: now also U14.3; no longer U65.6
- net ~{MEMOE}: now also U69.24 (~{OE})
- net ~{Mx}: no longer U31.14 (O1)
- net ~{Nx}: no longer U31.15 (O0)
- net ~{PUTO}: now also U51.1 (1OE), U51.19 (2OE); no longer U24.4, U74.12
- net ~{PUTR}: no longer U24.5
- net ~{RES}: now also U81.1 (~{Mr})
- net ~{RET}: now also U98.5 (UP)
- net ~{xD}: no longer U33.13 (O2)
- net ~{xM}: now also U14.4; no longer U24.3, U33.14 (O1)
- net at U37.11: now also U65.4, U75.1 (S)
- net at U38.2: now also U14.1; no longer U74.2
- net SUBR: now reaches U14.11, U37.4, U38.9
- net LO2: now reaches U79.12 (Zc), U85.14 (1Y2), U94.10 (A2)
- net LO2: now also U69.10 (A2)
- net LO1: now reaches U79.7 (Zb), U85.16 (1Y1), U94.11 (A1)
- net LO1: now also U69.11 (A1)
- net LO0: now reaches U79.4 (Za), U85.18 (1Y0), U94.12 (A0)
- net LO0: now also U69.12 (A0)
- net HI2: now reaches U94.23 (A10)
- net HI2: now also U62.14 (1Y2), U68.14 (1Y2), U69.23 (A10), U72.14 (1Y2)
- net HI3: now reaches U94.25 (A11)
- net HI3: now also U62.12 (1Y3), U68.12 (1Y3), U69.25 (A11), U72.12 (1Y3)
- net HI1: now reaches U94.26 (A9)
- net HI1: now also U62.16 (1Y1), U68.16 (1Y1), U69.26 (A9), U72.16 (1Y1)
- net HI0: now reaches U94.27 (A8)
- net HI0: now also U62.18 (1Y0), U68.18 (1Y0), U69.27 (A8), U72.18 (1Y0)
- net HI5: now reaches U94.28 (A13)
- net HI5: now also U62.5 (2Y1), U68.5 (2Y1), U69.28 (A13), U72.5 (2Y1)
- net HI4: now reaches U94.4 (A12)
- net HI4: now also U62.3 (2Y0), U68.3 (2Y0), U69.4 (A12), U72.3 (2Y0)
- net LO5: now reaches U78.7 (Zb), U85.5 (2Y1), U94.7 (A5)
- net LO5: now also U69.7 (A5)
- net LO4: now reaches U78.4 (Za), U85.3 (2Y0), U94.8 (A4)
- net LO4: now also U69.8 (A4)
- net LO3: now reaches U79.9 (Zd), U85.12 (1Y3), U94.9 (A3)
- net LO3: now also U69.9 (A3)
- net at U47.8: no longer U65.13
- net at U14.6: now also U69.29 (~{WE})
- net at U47.11: no longer U65.12
- net at U24.6: no longer U14.4
- net HI7: now reaches U14.2
- net HI7: now also U94.3 (A15), U62.9 (2Y3), U68.9 (2Y3), U69.31 (A15), U72.9 (2Y3); no longer U30.10
- net xLM_pre: now reaches U10.13 (Y2)
- net xLM_pre: now also U30.9
- net ~{GMacc}: now reaches U42.4
- net ~{GMacc}: now also U68.1 (1OE), U68.19 (2OE)
- net GorC: no longer names the net of U65.3
- net page_MSB: no longer names the net of U74.9
- net page_MSB: no longer U65.4
- net ~{GorL}: no longer names the net of U47.13
- net ~{GorL}: no longer U52.6
- net ~{Ox}: no longer names the net of U74.13
- net ~{Ox}: no longer U31.12 (O3)
- new net: U76.12 (Zd), U81.8 (D3)
- new net: U76.4 (Za), U81.3 (D0)
- new net: U76.7 (Zb), U81.4 (D1)
- new net: U76.9 (Zc), U81.7 (D2)
- new net: U62.4 (1A1), U98.2 (QB)
- new net: U62.2 (1A0), U98.3 (QA)
- new net: U62.6 (1A2), U98.6 (QC)
- new net: U62.8 (1A3), U98.7 (QD)
- new net: U75.12 (Zd), U81.18 (D7)
- new net: U75.4 (Za), U81.13 (D4)
- new net: U75.7 (Zb), U81.14 (D5)
- new net: U75.9 (Zc), U81.17 (D6)
- new net: U65.6, U81.11 (Cp)
- new net: U62.11 (2A3), U99.7 (QD)
- new net: U62.13 (2A2), U99.6 (QC)
- new net: U62.15 (2A1), U99.2 (QB)
- new net: U62.17 (2A0), U99.3 (QA)
- new net CMx_pre: U12.15 (Y0), U52.5
- new net GC_pre: U45.9
- new net GMx_pre: U12.14 (Y1), U42.5
- new net Gx: U30.12
- new net HI6: U62.7 (2Y2), U68.7 (2Y2), U69.3 (A14), U72.7 (2Y2), U94.29 (A14)
- new net LMx_pre: U12.13 (Y2), U30.8
- new net xGM_pre: U10.14 (Y1), U42.6
- new net ~{CMacc}: U52.6, U72.1 (1OE), U72.19 (2OE)
- new net ~{CMx}: U31.15 (O0)
- new net ~{GMx}: U31.14 (O1)
- new net ~{Gx}: U31.12 (O3)
- new net ~{LMacc}: U30.10, U38.1, U62.1 (1OE), U62.19 (2OE), U69.2 (A16)
- new net ~{LMx}: U31.13 (O2)
- new net ~{xGM}: U33.14 (O1)
- new net ~{xLM}: U33.13 (O2)
- no-connect marks 101 -> 97
Other:
- note added: "(CODE) Page index"
- note added: "(GLOBAL) Page index"
- note added: "(JUMP) register (Program Counter)"
- note added: "(LOCAL) Page index (Stack Pointer)"
- note added: "(OFFSET) Operand Register"
- note added: "(Relative addressing)"
- note added: "J does not get a new non-zero value during TRAP or CALL, it only gets zeroed; Execution starts at offset zero, the "head" of the destination page."
- note added: "L"
- note added: "When DC is executed, prevents the DB output from being updated with the new return address page index, before the instruction is done."
- note removed: "(8th bit selects RAM/ROM when not GorL)"
- note removed: "(DATA) Segment index"
- note removed: "(GLOBAL) Segment index"
- note removed: "(GorL = GLOBAL or LOCAL, including GETPUT)"
- note removed: "(Relative jumps)"
- note removed: "573 type TRANSPARENT latch"
- note removed: "7-BIT Page index"
- note removed: "C(ode) page index"
- note removed: "Conceptually, memory layout is: 128 (code/data) 64 (global) 64 (local) Physically, the layout is: 64 64 64 64"
- note removed: "D"
- note removed: "High"
- note removed: "Jump register (Program Counter)"
- note removed: "L (LOCAL) Segment index (Stack Pointer)"
- note removed: "O(rigin) Register"
- note removed: "Post-inc/dec on DATA RD/WR"
- note removed: "R new"
- note removed: "R old"
- note removed: "RAM 16k: 128 CODE/DATA pages @ 128 bytes 16k: (unused) 32k: 256 pairs of (Global + Local segments @ 64 bytes each)"
- note removed: "ROM 16k: 128 CODE/DATA pages @ 128 bytes"
- note removed: "Read data also when: GETPUT low and IB2 low (GET mode)"
- moved on the sheet: U13B, U14A, U15A, U15B, U1C, U24B, U25A, U25D, U28A, U30A, U30C, U30D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

Commit message: Remove offset-mapped segmentation
Parts:
- removed U24: 74HC11, Package_DIP:DIP-14_W7.62mm_Socket_LongPads, symbol 74xx:74LS11
- removed unit 1 of U25
- removed U65: 74HC32, Package_DIP:DIP-14_W7.62mm_Socket_LongPads, symbol 74xx:74LS32
- removed U69: 628128_DIP32_SSOP32, symbol Memory_RAM:628128_DIP32_SSOP32
- removed U74: 74LS08, Package_DIP:DIP-14_W7.62mm_Socket_LongPads, symbol 74xx:74LS08
- added unit 3 of U27
- added U59: KM62256CLP, Package_DIP:DIP-28_W15.24mm, symbol Memory_RAM:KM62256CLP
- renumbered U19 to U18, U18 to U19, U42 to U20, U30 to U21, U20 to U22, U21 to U23, U47 to U24, U22 to U25, U23 to U26, U25 to U27, U26 to U28, U27 to U29, U28 to U30, U29 to U31, U31 to U32, U32 to U33, U33 to U34, U34 to U35, U35 to U36, U36 to U37, U37 to U38, U38 to U39, U39 to U40, U75 to U41, U76 to U42, U40 to U43, U41 to U44, U81 to U45, U43 to U46, U46 to U47, U44 to U48, U51 to U49, U52 to U50, U45 to U51, U67 to U52, U48 to U53, U49 to U54, U50 to U55, U55 to U56, U56 to U57, U57 to U58, U58 to U60, U98 to U62, U99 to U63, U53 to U64, U54 to U65, U73 to U66, U63 to U67, U64 to U68, U62 to U69, U59 to U70, U60 to U71, U78 to U72, U79 to U73, U70 to U74, U71 to U75, U85 to U76, U88 to U78, U89 to U79, U82 to U80, U83 to U81, U84 to U82, U72 to U83, U66 to U84, U92 to U85, U94 to U87, U68 to U88
Connections:
- net DC_pre is gone; now on net GC_pre: U15.8
- net Dx is gone; now on net Gx: U50.8
- net GLOBAL is gone; now on an unnamed net: U38.8
- net Mx_pre is gone; now on net GMx_pre: U5.5
- net xA is gone; now on net GND: U39.5
- net xM_pre is gone; now on net xGM_pre: U5.2, U5.4
- net ~{CMx} is gone; now on net ~{Nx}: U32.15 (O0)
- net ~{Dx} is gone; now on net ~{Gx}: U50.9
- net ~{Mx} is gone; now on net ~{GMx}: U47.11
- net ~{xD} is gone; now on net ~{GETR}: U50.1
- net ~{xM} is gone; now on an unnamed net: U14.4
- net +5V: now also U59.28 (VCC); no longer U62.1 (B), U62.10 (C), U62.11 (~{LOAD}), U62.15 (A), U62.9 (D), U63.1 (B), U63.10 (C), U63.11 (~{LOAD}), U63.15 (A), U63.9 (D)
- net DB0: now also U62.15 (A), U59.11 (Q0)
- net DB1: now also U62.1 (B), U59.12 (Q1)
- net DB2: now also U62.10 (C), U59.13 (Q2)
- net DB3: now also U62.9 (D), U59.15 (Q3)
- net DB4: now also U63.15 (A), U59.16 (Q4)
- net DB5: now also U63.1 (B), U59.17 (Q5)
- net DB6: now also U63.10 (C), U59.18 (Q6)
- net DB7: now also U63.9 (D), U59.19 (Q7)
- net FETCH: now also U13.12; no longer U1.9
- net GETO: now also U27.9
- net GETPUT: no longer U15.5
- net GND: now also U1.8, U1.9, U14.2, U15.12, U15.13, U15.4, U15.5, U24.1, U24.2, U24.4, U24.5, U39.1, U4.3, U87.3 (A15); no longer U44.10, U44.12, U44.13, U44.9
- net HI0: now also U59.25 (A8)
- net HI1: now also U59.24 (A9)
- net HI2: now also U59.21 (A10)
- net HI3: now also U59.23 (A11)
- net HI4: now also U59.2 (A12)
- net HI5: now also U59.26 (A13)
- net HI6: now also U59.1 (A14)
- net HI7: now also U51.1, U87.22 (CE); no longer U14.2, U87.3 (A15)
- net IB2: no longer U15.4
- net IPH: now also U20.9
- net J0: now also U67.5 (A1)
- net J1: now also U67.3 (A2)
- net J2: now also U67.14 (A3)
- net J3: now also U67.12 (A4)
- net J4: now also U67.6 (B1)
- net J5: now also U67.2 (B2)
- net J6: now also U67.15 (B3)
- net J7: now also U67.11 (B4)
- net JIN0: no longer U67.5 (A1)
- net JIN1: no longer U67.3 (A2)
- net JIN2: no longer U67.14 (A3)
- net JIN3: no longer U67.12 (A4)
- net JIN4: no longer U67.6 (B1)
- net JIN5: no longer U67.2 (B2)
- net JIN6: no longer U67.15 (B3)
- net JIN7: no longer U67.11 (B4)
- net LFETCH: now also U24.8
- net LO0: now also U59.10 (A0)
- net LO1: now also U59.9 (A1)
- net LO2: now also U59.8 (A2)
- net LO3: now also U59.7 (A3)
- net LO4: now also U59.6 (A4)
- net LO5: now also U59.5 (A5)
- net LO6: now also U59.4 (A6); no longer U47.13
- net LO7: now also U59.3 (A7); no longer U24.2
- net Nx_pre: now also U12.15 (Y0), U24.13
- net PH1: now also U24.9
- net SUBR: now also U38.10
- net xC_pre: no longer U15.13
- net ~{CMacc}: now also U20.10; no longer U50.6
- net ~{GETPUT}: no longer U24.1
- net ~{IN_RAM}: now also U59.20 (~{CS})
- net ~{LMacc}: no longer U39.1
- net ~{LMx}: now also U50.5
- net ~{MEMOE}: now also U13.13, U59.22 (~{OE}); no longer U1.10
- net ~{PUTO}: now also U44.9
- net ~{PUTR}: now also U44.10
- net ~{opc_ALU}: no longer U4.3
- net ~{xGM}: now also U44.13
- net ~{xLM}: now also U44.12, U50.3
- net at U24.6: no longer U38.10
- net at U38.9: now also U38.11, U41.1 (S), U42.1 (S); no longer U15.6
- net ~{xL}: now reaches U47.12
- net ~{xL}: now also U62.11 (~{LOAD}), U63.11 (~{LOAD}); no longer U24.5
- net at U24.3: no longer U24.4
- net at U18.12: now also U24.12
- net at U24.10: now also U20.8, U24.11
- net xL: now reaches U33.14 (Y1)
- net xL: now also U47.13
- net at U14.6: now also U59.27 (~{WE})
- net xLM: now reaches U50.4
- net LMx: now reaches U13.10
- net LMx: now also U50.6
- net GMx: now reaches U13.11
- net GMx: now also U47.10
- net at U13.9: now also U27.8
- removed net CMx_pre: U12.15 (Y0), U50.5
- net Dx_pre renamed Gx_pre
- net Gx_pre: now also U12.12 (Y3)
- removed net Mx: U1.8, U47.10
- net OC_pre: no longer names the net of U15.11
- removed net Ox_pre: U12.12 (Y3), U15.12
- net opc_ALU: no longer names the net of U4.4
- net xD renamed GETR
- net GETR: now also U27.10
- removed net ~{IN_ROM}: U14.3, U51.1, U87.22 (CE)
- net ~{xA}: no longer names the net of U39.6
- no-connect marks 97 -> 101
Other:
- note added: "HI7 switches between RAM and ROM"
- note added: "J (the program counter) is cleared/set to 0 during TRAP or CALL. Execution starts at offset zero, the "head" of the destination page."
- note added: "O provides the return offset during RET receives the return offset during SUBR can be GET and PUT provides all address offsets except FETCH can be stored into is the implied 2nd ALU input operand"
- note removed: "EITHER two contiguous 64 byte segments if offset between 0 and 127 and not GETPUT. OR ELSE GLOBAL or LOCAL 64 byte segment"
- note removed: "IF GETPUT: IB2 set = GLOBAL IB2 clear = LOCAL"
- note removed: "IF NOT GETPUT but LO7: LO6 set = LOCAL LO6 clear = GLOBAL"
- note removed: "J does not get a new non-zero value during TRAP or CALL, it only gets zeroed; Execution starts at offset zero, the "head" of the destination page."
- moved on the sheet: U13B, U14A, U15B, U15D, U18F, U1C, U20B, U20C, U21C, U24A, U24B, U24C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

Commit message: Fix the schematics
Parts:
- added unit 1 of U27
- renumbered U60 to U59, U61 to U60, U62 to U61, U63 to U62, U64 to U63, U65 to U64, U66 to U65, U67 to U66, U68 to U67, U69 to U68, U70 to U69, U71 to U70, U72 to U71, U73 to U72, U74 to U73, U75 to U74, U76 to U75, U77 to U76, U78 to U77, U79 to U78, U80 to U79, U81 to U80, U82 to U81, U83 to U82, U84 to U83, U85 to U84, U59 to U85, U87 to U86, U88 to U87
Connections:
- net GETO: no longer U27.9
- net GND: now also U50.1, U50.13, U50.3, U85.14 (GND), U27.1, U27.2; no longer U14.2, U39.1, U39.5, U40.1, U40.2
- net RET: now also U27.9; no longer U21.11, U38.5
- net SUBR: now also U14.2, U30.1; no longer U38.10
- net TRAP: no longer U30.1
- net xC: no longer U30.2
- net xG: now also U30.2; no longer U30.8
- net xO: now also U33.14 (Y1); no longer U50.12
- net xW_pre: now also U11.11 (Y4); no longer U11.12 (Y3)
- net ~{GETO}: now also U40.1
- net ~{GETR}: now also U40.2; no longer U50.1
- net ~{RET}: no longer U15.1
- net ~{xG}: now also U34.12 (O3); no longer U34.15 (O0)
- net ~{xLM}: no longer U50.3
- net ~{xL}: now also U34.15 (O0); no longer U47.12
- net BRA: now reaches U39.6
- net BRA: now also U27.10
- net HERE: now reaches U14.1, U39.2
- net ~{HERE}: now reaches U25.7 (O7)
- net ~{HERE}: now also U30.8, U39.1
- net ~{BRA}: now reaches U25.9 (O6)
- net ~{BRA}: now also U39.5
- net at U13.9: now also U40.3; no longer U27.8
- net at U14.3: now also U38.10
- net GETR: no longer names the net of U50.2
- net GETR: no longer U27.10
- net xL renamed RETBRA
- net RETBRA: now also U21.11, U27.8, U38.5; no longer U33.14 (Y1)
- net xLM: no longer names the net of U50.4
- removed net ~{xO}: U34.12 (O3), U50.13
- new net: U15.1, U47.12
- no-connect marks 101 -> 99
Other:
- note added: "IN_ROM"
- moved on the sheet: U14A, U15D, U1C, U27C, U39A, U39C, U40A, U47F, U4D, U50A, U50B, U50F
