File: Schematics/myth.kicad_sch (KiCad schematic)
At the start: 128 parts, among them J1 Conn_01x08_Male, J2 Conn_01x08_Male, J3 Conn_01x08_Male, J4 Conn_01x08_Male, J5 Conn_01x04_Male, J6 Conn_01x04_Male, J7 Conn_02x01, U1 74AHC02, U10 74HC595, U11 74HC165, U12 74AHC08, U13 74HC238, U14 74HC238, U15 74HC238, U16 4002, U17 74HC32, U18 74AHC273, U19 CD4532BE, U2 74AHC273, U20 74AHC138, U21 74AHC04, U22 74AHC138, U23 74LS32, U24 74HC238, U25 74HC238, U26 4078, U27 74AHC244, U28 74AHC138, U29 74AHC138, U3 74HC74, U30 4075, U31 74AHC02, U32 74AHC138, U33 74HC238, U34 74AHC138, U35 74HC163, U36 74AHC574, U37 74HC238, U38 74HC32, U39 74AHC04, U4 74AHC04, U40 74HC00, U41 74AHC574, U42 74HC74, U43 74AHC273, U44 74HC283, U45 74HC283, U46 74AHC273, U47 74HC02, U48 74HC157, U49 74HC157, U5 74AHC04, U50 74AHC244, U51 74AHC04, U52 74LS32, U53 74AHC574, U55 74HC193, U56 74HC193, U57 74HC193, U58 74HC193, U59 74HC193, U6 74AHC08, U60 74HC193, U61 74AHC244, U62 4078, U63 74LS21, U64 74AHC04, U65 74AHC244, U66 74AHC273, U67 74HC157, U68 74HC157, U69 74HC157, U7 74LS08, U70 74HC157, U71 74LS257, U72 74LS257, U73 74AHC273, U74 74AHC273, U75 74AHC244, U76 74AHC574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

Commit message: Clean up the schematics
Parts:
- removed U7: 74LS08, Package_DIP:DIP-14_W7.62mm_Socket_LongPads, symbol 74xx:74LS08
- removed U76: 74AHC574, Package_DIP:DIP-20_W7.62mm_Socket_LongPads, symbol 74xx:74LS574
- added J1, J4, J5, J7: Conn_01x08_Male, Connector_PinHeader_2.54mm:PinHeader_1x08_P2.54mm_Vertical, symbol Connector:Conn_01x08_Male
- added U57: 74AHC273, Package_DIP:DIP-20_W7.62mm_Socket_LongPads, symbol 74xx:74HC273
- added U77: 74AHC244, Package_DIP:DIP-20_W7.62mm_Socket_LongPads, symbol 74xx:74AHC244
- renumbered J6 to J10, J7 to J11, J1 to J2, J2 to J3, J3 to J6, J4 to J8, J5 to J9, U52 to U19, U19 to U20, U20 to U21, U21 to U22, U22 to U23, U23 to U26, U26 to U27, U27 to U28, U28 to U29, U29 to U30, U30 to U31, U31 to U32, U32 to U33, U33 to U34, U34 to U35, U35 to U36, U36 to U37, U37 to U38, U38 to U39, U39 to U40, U53 to U52, U55 to U53, U56 to U54, U57 to U55, U58 to U56, U59 to U58, U60 to U59, U61 to U60, U91 to U61, U65 to U63, U63 to U64, U64 to U65, U40 to U7, U77 to U76
Connections:
- net +5V: now also U57.20 (VCC), U77.20 (VCC)
- net D0: now also U77.2 (1A0)
- net D1: now also U77.4 (1A1)
- net D2: now also U77.6 (1A2)
- net D3: now also U77.8 (1A3)
- net D4: now also U77.17 (2A0)
- net D5: now also U77.15 (2A1)
- net D6: now also U77.13 (2A2)
- net D7: now also U77.11 (2A3)
- net DB0: now also U57.3 (D0), U77.18 (1Y0)
- net DB1: now also U57.4 (D1), U77.16 (1Y1)
- net DB2: now also U57.7 (D2), U77.14 (1Y2)
- net DB3: now also U57.8 (D3), U77.12 (1Y3)
- net DB4: now also U57.13 (D4), U77.3 (2Y0)
- net DB5: now also U57.14 (D5), U77.5 (2Y1)
- net DB6: now also U57.17 (D6), U77.7 (2Y2)
- net DB7: now also U57.18 (D7), U77.9 (2Y3)
- net DH10: now also J5.1 (Pin_1)
- net DH11: now also J5.2 (Pin_2)
- net DH12: now also J5.3 (Pin_3)
- net DH13: now also J5.4 (Pin_4)
- net DH14: now also J5.5 (Pin_5)
- net DH15: now also J5.6 (Pin_6)
- net DH2: now also J6.1 (Pin_1)
- net DH3: now also J6.2 (Pin_2)
- net DH4: now also J6.3 (Pin_3)
- net DH5: now also J6.4 (Pin_4)
- net DH6: now also J6.5 (Pin_5)
- net DH7: now also J6.6 (Pin_6)
- net DH8: now also J6.7 (Pin_7)
- net DH9: now also J6.8 (Pin_8)
- net EH0: no longer J6.1 (Pin_1)
- net EH1: no longer J6.2 (Pin_2)
- net EH2: no longer J6.3 (Pin_3)
- net EH3: no longer J6.4 (Pin_4)
- net EL0: no longer J6.5 (Pin_5)
- net EL1: no longer J6.6 (Pin_6)
- net EL2: no longer J6.7 (Pin_7)
- net EL3: no longer J6.8 (Pin_8)
- net GND: now also U61.10, U61.9, U57.10 (GND), U77.10 (GND); no longer U47.2, U47.3, U8.1, U8.2
- net PUTD: now also U32.12; no longer U61.9
- net xB: now also U57.11 (Cp)
- net ~{DL10}: now also J4.8 (Pin_8)
- net ~{DL11}: now also J4.7 (Pin_7)
- net ~{DL12}: now also J4.6 (Pin_6)
- net ~{DL13}: now also J4.5 (Pin_5)
- net ~{DL14}: now also J4.4 (Pin_4)
- net ~{DL15}: now also J4.3 (Pin_3)
- net ~{DL2}: now also J1.8 (Pin_8)
- net ~{DL3}: now also J1.7 (Pin_7)
- net ~{DL4}: now also J1.6 (Pin_6)
- net ~{DL5}: now also J1.5 (Pin_5)
- net ~{DL6}: now also J1.4 (Pin_4)
- net ~{DL7}: now also J1.3 (Pin_3)
- net ~{DL8}: now also J1.2 (Pin_2)
- net ~{DL9}: now also J1.1 (Pin_1)
- net ~{RES}: now also U57.1 (~{Mr})
- net at U55.11 (~{LOAD}), U56.11 (~{LOAD}): now also U8.3
- net at U51.12: now also U8.1
- net PUTG: now reaches U65.8
- net PUTG: now also U47.2
- net at U47.1: now also U52.1 (OE)
- net at U61.8: no longer U32.12
- net at U32.13: now also U77.1 (1OE), U77.19 (2OE)
- net at U7.11: now also U8.2
- net DC_pre renamed ~{PUTG}
- net ~{PUTG}: now also U9.7 (O7)
- net Dx renamed Gx
- net Gx: now also U47.3; no longer U61.10
- net Dx_pre: no longer names the net of U15.12 (Y3)
- net GETA renamed GETG
- net xA renamed xG
- net xC_pre: no longer names the net of U14.7 (Y7)
- net ~{Dx} renamed ~{Gx}
- net ~{GETA} renamed ~{GETG}
- removed net ~{PUTA}: U52.1 (OE), U9.7 (O7)
- new net B0: J7.8 (Pin_8), U57.2 (Q0)
- new net B1: J7.7 (Pin_7), U57.5 (Q1)
- new net B2: J7.6 (Pin_6), U57.6 (Q2)
- new net B3: J7.5 (Pin_5), U57.9 (Q3)
- new net B4: J7.4 (Pin_4), U57.12 (Q4)
- new net B5: J7.3 (Pin_3), U57.15 (Q5)
- new net B6: J7.2 (Pin_2), U57.16 (Q6)
- new net B7: J7.1 (Pin_1), U57.19 (Q7)
- no-connect marks 91 -> 65
Other:
- note added: "(BROADCAST)"
- note added: "(GLOBAL)"
- note added: "B"
- note added: "Core Intent Broadcast"
- note added: "Currently mapped to NOP, reserved for instruction set extensions"
- note added: "G"
- note added: "Internal data bus header"
- note added: "R/O/D/G"
- note added: "Remap ("scrounge") MM, RR, DD etc, and impracticable opcodes such as NM"
- note added: "etc."
- note removed: "(A spare register)"
- note removed: "A"
- note removed: "Anything"
- note removed: "Broadcast"
- note removed: "Currently NOP, reserved for instruction set extension"
- note removed: "Etc."
- note removed: "R/O/G/A"
- note removed: "Remap MM, RR, DD etc, and impracticable opcodes such as NM"
- moved on the sheet: RN1, RN2, U18, U19A, U1C, U24, U25, U26A, U29, U30, U31A, U32D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

Commit message: Add schematics
Connections:
- net xD: now also U34.13 (Y2); no longer U22.10
- net xE: now also U34.15 (Y0); no longer U34.13 (Y2)
- net xG: now also U22.10; no longer U34.15 (Y0)
- net ~{xD} renamed ~{xG}
Changed lines of the file:
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@@
 	(title_block
 		(title "Sonne-8 Micro-Controller")
-		(date "2024-08-17")
+		(date "2024-08-18")
 		(rev "Myth Kelvin")
 		(company "Contact: mim@ok-schalter.de")
@@
 	)
 	(label "xE"
-		(at 364.9218 307.0098 0)
+		(at 364.9218 301.9298 0)
 		(fields_autoplaced yes)
 		(effects
@@
 		)
 	)
-	(label "xD"
-		(at 719.535 218.2954 0)
+	(label "~{xG}"
+		(at 704.295 218.2954 180)
 		(fields_autoplaced yes)
 		(effects
@@
 				(size 1.27 1.27)
 			)
-			(justify left bottom)
+			(justify right bottom)
 		)
 	)
@@
 		)
 	)
-	(label "~{xD}"
-		(at 704.295 218.2954 180)
+	(label "xG"
+		(at 719.535 218.2954 0)
 		(fields_autoplaced yes)
 		(effects
@@
 				(size 1.27 1.27)
 			)
-			(justify right bottom)
+			(justify left bottom)
 		)
 	)
@@
 		)
 	)
-	(label "~{xD}"
-		(at 364.2868 271.4498 0)
+	(label "xD"
+		(at 364.9218 307.0098 0)
 		(fields_autoplaced yes)
 		(effects
@@
 		)
 	)
-	(label "xG"
-		(at 364.9218 301.9298 0)
+	(label "~{xG}"
+		(at 364.2868 271.4498 0)
 		(fields_autoplaced yes)
 		(effects

Commit message: Rename BRA opcode FAR
Connections:
- net BRA renamed FAR
- net RETBRA renamed RETFAR
- net ~{BRA} renamed ~{FAR}
Changed lines of the file:
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@@
 	(wire
 		(pts
-			(xy 921.7837 679.7257) (xy 924.3237 679.7257)
-		)
-		(stroke
-			(width 0)
-			(type default)
-		)
-	)
-	(wire
-		(pts
 			(xy 969.4592 141.7148) (xy 952.4412 141.7148)
 		)
@@
 		)
 	)
-	(label "BRA"
+	(label "FAR"
 		(at 375.6921 223.5482 180)
 		(fields_autoplaced yes)
@@
 		)
 	)
-	(label "~{BRA}"
+	(label "~{FAR}"
 		(at 744.0059 333.3548 180)
 		(fields_autoplaced yes)
@@
 		)
 	)
-	(label "RETBRA"
+	(label "RETFAR"
 		(at 921.7837 684.8057 0)
 		(fields_autoplaced yes)
@@
 		)
 	)
-	(label "RETBRA"
+	(label "RETFAR"
 		(at 394.0556 221.0082 0)
 		(fields_autoplaced yes)
@@
 		)
 	)
-	(label "BRA"
+	(label "FAR"
 		(at 759.2459 333.3548 0)
 		(fields_autoplaced yes)
@@
 	)
 	(label "PUTD"
-		(at 924.3119 679.7257 0)
+		(at 921.7837 679.7257 0)
 		(fields_autoplaced yes)
 		(effects
@@
 		)
 	)
-	(label "RETBRA"
+	(label "RETFAR"
 		(at 558.7035 328.2623 180)
 		(fields_autoplaced yes)
@@
 		)
 	)
-	(label "~{BRA}"
+	(label "~{FAR}"
 		(at 216.6174 390.1948 0)
 		(fields_autoplaced yes)

Commit message: Rename B register, change functionality of it
Parts:
- removed J7: Conn_01x08_Male, Connector_PinHeader_2.54mm:PinHeader_1x08_P2.54mm_Vertical, symbol Connector:Conn_01x08_Male
- removed U57: 74AHC273, Package_DIP:DIP-20_W7.62mm_Socket_LongPads, symbol 74xx:74HC273
- added U91, U92: 74HC283, Package_DIP:DIP-16_W7.62mm_Socket_LongPads, symbol 74xx:74LS283
- added U93, U94: 74HC157, Package_DIP:DIP-16_W7.62mm_Socket_LongPads, symbol 74xx:74LS157
Connections:
- net +5V: now also U91.16 (VCC), U92.16 (VCC), U93.16 (VCC), U94.16 (VCC)
- net DB0: now also U91.6 (B1), U93.2 (I0a); no longer U52.2 (D0)
- net DB1: now also U91.2 (B2), U93.5 (I0b); no longer U52.3 (D1)
- net DB2: now also U91.15 (B3), U93.11 (I0c); no longer U52.4 (D2)
- net DB3: now also U91.11 (B4), U93.14 (I0d); no longer U52.5 (D3)
- net DB4: now also U92.6 (B1), U94.2 (I0a); no longer U52.6 (D4)
- net DB5: now also U92.2 (B2), U94.5 (I0b); no longer U52.7 (D5)
- net DB6: now also U92.15 (B3), U94.11 (I0c); no longer U52.8 (D6)
- net DB7: now also U92.11 (B4), U94.14 (I0d); no longer U52.9 (D7)
- net GETG: now also U26.2; no longer U26.1
- net GND: now also U91.7 (C0), U91.8 (GND), U92.8 (GND), U93.15 (E), U93.8 (GND), U94.15 (E), U94.8 (GND); no longer U61.1, U61.2
- net I0: now also U91.5 (A1)
- net I1: now also U91.3 (A2)
- net I2: now also U91.14 (A3)
- net I3: now also U91.12 (A4)
- net I4: now also U92.5 (A1)
- net I5: now also U92.3 (A2)
- net I6: now also U92.14 (A3)
- net I7: now also U92.12 (A4)
- net xG: now also U61.1; no longer U26.2
- net at U61.3: now also U26.1
- net xB renamed xA
- net xA: now also U61.2, U93.1 (S), U94.1 (S)
- new net: U91.1 (S2), U93.6 (I1b)
- new net: U91.10 (S4), U93.13 (I1d)
- new net: U91.13 (S3), U93.10 (I1c)
- new net: U91.4 (S1), U93.3 (I1a)
- new net: U91.9 (C4), U92.7 (C0)
- new net: U92.1 (S2), U94.6 (I1b)
- new net: U92.10 (S4), U94.13 (I1d)
- new net: U92.13 (S3), U94.10 (I1c)
- new net: U92.4 (S1), U94.3 (I1a)
- new net GIN0: U52.2 (D0), U93.4 (Za)
- new net GIN1: U52.3 (D1), U93.7 (Zb)
- new net GIN2: U52.4 (D2), U93.9 (Zc)
- new net GIN3: U52.5 (D3), U93.12 (Zd)
- new net GIN4: U52.6 (D4), U94.4 (Za)
- new net GIN5: U52.7 (D5), U94.7 (Zb)
- new net GIN6: U52.8 (D6), U94.9 (Zc)
- new net GIN7: U52.9 (D7), U94.12 (Zd)
Other:
- note added: "ADD i"
- note added: "Load DB value (xG) or DB + I (xA = "ADD")"
- note removed: "(BROADCAST)"
- note removed: "B"
- note removed: "Core Intent Broadcast"
- moved on the sheet: U26A, U47A, U52, U61A

Commit message: Add groff doc source
Connections:
- net DH10 renamed SH10
- net DH11 renamed SH11
- net DH12 renamed SH12
- net DH13 renamed SH13
- net DH14 renamed SH14
- net DH15 renamed SH15
- net DH2 renamed SH2
- net DH3 renamed SH3
- net DH4 renamed SH4
- net DH5 renamed SH5
- net DH6 renamed SH6
- net DH7 renamed SH7
- net DH8 renamed SH8
- net DH9 renamed SH9
- net ~{DL10} renamed ~{SL10}
- net ~{DL11} renamed ~{SL11}
- net ~{DL12} renamed ~{SL12}
- net ~{DL13} renamed ~{SL13}
- net ~{DL14} renamed ~{SL14}
- net ~{DL15} renamed ~{SL15}
- net ~{DL2} renamed ~{SL2}
- net ~{DL3} renamed ~{SL3}
- net ~{DL4} renamed ~{SL4}
- net ~{DL5} renamed ~{SL5}
- net ~{DL6} renamed ~{SL6}
- net ~{DL7} renamed ~{SL7}
- net ~{DL8} renamed ~{SL8}
- net ~{DL9} renamed ~{SL9}
Other:
- note added: "Jump while value register I not zero (decrements I)"
- note removed: "Jump while value register V not zero (decrements V)"
Changed lines of the file:
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@@
 		)
 	)
-	(text "Jump while value register V not zero\n(decrements V)"
+	(text "Jump while value register I not zero\n(decrements I)"
 		(exclude_from_sim no)
 		(at 65.8996 179.5348 0)
@@
 		)
 	)
-	(label "~{DL4}"
+	(label "~{SL4}"
 		(at 120.707 112.5444 180)
 		(fields_autoplaced yes)
@@
 		)
 	)
+	(label "IB5"
+		(at 169.9205 496.4938 180)
+		(fields_autoplaced yes)
+		(effects
+			(font
+				(size 1.27 1.27)
+			)
+			(justify right bottom)
+		)
+	)
 	(label "+5V"
 		(at 376.047 71.7296 180)
@@
 		)
 	)
-	(label "~{DL9}"
+	(label "~{SL9}"
 		(at 120.707 125.2444 180)
 		(fields_autoplaced yes)
@@
 		)
 	)
-	(label "~{DL3}"
+	(label "~{SL3}"
 		(at 120.707 110.0044 180)
 		(fields_autoplaced yes)
@@
 		)
 	)
-	(label "DH15"
+	(label "SH15"
 		(at 262.7715 741.6931 0)
 		(fields_autoplaced yes)
@@
 		)
 	)
-	(label "~{DL9}"
+	(label "~{SL9}"
 		(at 309.1071 736.8894 0)
 		(fields_autoplaced yes)
@@
 		)
 	)
-	(label "DH7"
+	(label "SH7"
 		(at 262.5131 702.8138 0)
 		(fields_autoplaced yes)
@@
 		)
 	)
-	(label "~{DL12}"
+	(label "~{SL12}"
 		(at 309.1071 744.5094 0)
 		(fields_autoplaced yes)
@@
 		)
 	)
-	(label "~{DL3}"
+	(label "~{SL3}"
 		(at 308.966 692.8498 0)
 		(fields_autoplaced yes)
@@
 		)
 	)
-	(label "~{DL13}"
+	(label "~{SL13}"
 		(at 148.2648 117.873 0)
 		(fields_autoplaced yes)
@@
 		)
 	)
-	(label "DH5"
+	(label "SH5"
 		(at 148.4122 61.3156 0)
 		(fields_autoplaced yes)
@@
 		)
 	)
-	(label "~{DL6}"
+	(label "~{SL6}"
 		(at 120.707 117.6244 180)
 		(fields_autoplaced yes)
@@
 		)
 	)
-	(label "~{DL10}"
+	(label "~{SL10}"
 		(at 309.1071 739.4294 0)
 		(fields_autoplaced yes)
@@
 		)
 	)
-	(label "~{DL8}"
+	(label "~{SL8}"
 		(at 309.1071 734.3494 0)
 		(fields_autoplaced yes)
@@
 		)
 	)
-	(label "DH3"
+	(label "SH3"
 		(at 262.5131 692.6538 0)
 		(fields_autoplaced yes)
@@
 		)
 	)
-	(label "~{DL2}"
+	(label "~{SL2}"
 		(at 120.707 107.4644 180)
 		(fields_autoplaced yes)
@@
 		)
 	)
-	(label "~{DL5}"
+	(label "~{SL5}"
 		(at 120.707 115.0844 180)
 		(fields_autoplaced yes)
@@
 		)
 	)
-	(label "~{DL8}"
+	(label "~{SL8}"
 		(at 120.707 122.7044 180)
 		(fields_autoplaced yes)
@@
 		)
 	)
-	(label "DH8"
+	(label "SH8"
 		(at 148.4122 68.9356 0)
 		(fields_autoplaced yes)
@@
 		)
 	)
+	(label "IB7"
+		(at 169.7912 501.5738 180)
+		(fields_autoplaced yes)
+		(effects
+			(font
+				(size 1.27 1.27)
+			)
+			(justify right bottom)
+		)
+	)
 	(label "EL1"
 		(at 283.566 687.7698 180)
@@
 		)
 	)
-	(label "~{DL12}"
+	(label "~{SL12}"
 		(at 148.2648 120.413 0)
 		(fields_autoplaced yes)
@@
 		)
 	)
-	(label "DH2"
+	(label "SH2"
 		(at 148.4122 53.6956 0)
 		(fields_autoplaced yes)
@@
 		)
 	)
-	(label "~{DL14}"
+	(label "IB3"
+		(at 173.0455 491.4138 180)
+		(fields_autoplaced yes)
+		(effects
+			(font
+				(size 1.27 1.27)
+			)
+			(justify right bottom)
+		)
+	)
+	(label "~{SL14}"
 		(at 148.2648 115.333 0)
 		(fields_autoplaced yes)
@@
 		)
 	)
-	(label "~{DL4}"
+	(label "~{SL4}"
 		(at 308.966 695.3898 0)
 		(fields_autoplaced yes)
@@
 		)
 	)
-	(label "DH15"
+	(label "SH15"
 		(at 148.3259 91.1631 0)
 		(fields_autoplaced yes)
@@
 		)
 	)
-	(label "DH5"
+	(label "SH5"
 		(at 262.5131 697.7338 0)
 		(fields_autoplaced yes)
@@
 		)
 	)
-	(label "DH6"
+	(label "SH6"
 		(at 148.4122 63.8556 0)
 		(fields_autoplaced yes)
@@
 		)
 	)
+	(label "IB6"
+		(at 169.7763 499.0338 180)
+		(fields_autoplaced yes)
+		(effects
+			(font
+				(size 1.27 1.27)
+			)
+			(justify right bottom)
+		)
+	)
 	(label "J2"
 		(at 645.0549 350.0631 0)
@@
 		)
 	)
-	(label "~{DL5}"
+	(label "~{SL5}"
 		(at 308.966 697.9298 0)
 		(fields_autoplaced yes)
@@
 		)
 	)
-	(label "~{DL15}"
+	(label "~{SL15}"
 		(at 309.1071 752.1294 0)
 		(fields_autoplaced yes)
@@
 		)
 	)
-	(label "DH2"
+	(label "SH2"
 		(at 262.5131 690.1138 0)
 		(fields_autoplaced yes)
@@
 		)
 	)
-	(label "DH13"
+	(label "SH13"
 		(at 148.3259 86.0831 0)
 		(fields_autoplaced yes)
@@
 		)
 	)
-	(label "~{DL2}"
+	(label "~{SL2}"
 		(at 308.966 690.3098 0)
 		(fields_autoplaced yes)
@@
 		)
 	)
-	(label "DH3"
+	(label "SH3"
 		(at 148.4122 56.2356 0)
 		(fields_autoplaced yes)
@@
 		)
 	)
-	(label "~{DL11}"
+	(label "~{SL11}"
 		(at 309.1071 741.9694 0)
 		(fields_autoplaced yes)
@@
 		)
 	)
-	(label "DH8"
+	(label "SH8"
 		(at 262.7715 723.9131 0)
 		(fields_autoplaced yes)
@@
 		)
 	)
-	(label "DH11"
+	(label "SH11"
 		(at 148.3259 81.0031 0)
 		(fields_autoplaced yes)
@@
 		)
 	)
-	(label "~{DL11}"
+	(label "~{SL11}"
 		(at 148.2648 122.953 0)
 		(fields_autoplaced yes)
@@
 		)
 	)
-	(label "DH9"
+	(label "SH9"
 		(at 148.4122 71.4756 0)
 		(fields_autoplaced yes)
@@
 		)
 	)
-	(label "DH7"
+	(label "SH7"
 		(at 148.4122 66.3956 0)
 		(fields_autoplaced yes)
@@
 		)
 	)
-	(label "DH10"
+	(label "SH10"
 		(at 148.3259 78.4631 0)
 		(fields_autoplaced yes)
@@
 		)
 	)
-	(label "~{DL6}"
+	(label "~{SL6}"
 		(at 308.966 700.4698 0)
 		(fields_autoplaced yes)
@@
 		)
 	)
-	(label "DH11"
+	(label "SH11"
 		(at 262.7715 731.5331 0)
 		(fields_autoplaced yes)
@@
 		)
 	)
-	(label "DH13"
+	(label "SH13"
 		(at 262.7715 736.6131 0)
 		(fields_autoplaced yes)
@@
 		)
 	)
-	(label "~{DL13}"
+	(label "~{SL13}"
 		(at 309.1071 747.0494 0)
 		(fields_autoplaced yes)
@@
 		)
 	)
-	(label "~{DL7}"
+	(label "~{SL7}"
 		(at 120.707 120.1644 180)
 		(fields_autoplaced yes)
@@
 		)
 	)
-	(label "DH4"
+	(label "SH4"
 		(at 148.4122 58.7756 0)
 		(fields_autoplaced yes)
@@
 		)
 	)
-	(label "DH14"
+	(label "SH14"
 		(at 262.7715 739.1531 0)
 		(fields_autoplaced yes)
@@
 		)
 	)
-	(label "DH10"
+	(label "SH10"
 		(at 262.7715 728.9931 0)
 		(fields_autoplaced yes)
@@
 		)
 	)
-	(label "~{DL14}"
+	(label "~{SL14}"
 		(at 309.1071 749.5894 0)
 		(fields_autoplaced yes)
@@
 		)
 	)
-	(label "~{DL15}"
+	(label "~{SL15}"
 		(at 148.2648 112.793 0)
 		(fields_autoplaced yes)
@@
 		)
 	)
-	(label "~{DL10}"
+	(label "~{SL10}"
 		(at 148.2648 125.493 0)
 		(fields_autoplaced yes)
@@
 		)
 	)
+	(label "IB4"
+		(at 171.0263 493.9538 180)
+		(fields_autoplaced yes)
+		(effects
+			(font
+				(size 1.27 1.27)
+			)
+			(justify right bottom)
+		)
+	)
 	(label "HI2"
 		(at 1000.9648 557.1564 180)
@@
 		)
 	)
-	(label "DH12"
+	(label "SH12"
 		(at 262.7715 734.0731 0)
 		(fields_autoplaced yes)
@@
 		)
 	)
-	(label "DH12"
+	(label "SH12"
 		(at 148.3259 83.5431 0)
 		(fields_autoplaced yes)
@@
 		)
 	)
-	(label "DH6"
+	(label "SH6"
 		(at 262.5131 700.2738 0)
 		(fields_autoplaced yes)
@@
 		)
 	)
-	(label "DH14"
+	(label "SH14"
 		(at 148.3259 88.6231 0)
 		(fields_autoplaced yes)
@@
 		)
 	)
-	(label "~{DL7}"
+	(label "~{SL7}"
 		(at 308.966 703.0098 0)
 		(fields_autoplaced yes)
@@
 		)
 	)
-	(label "DH9"
+	(label "SH9"
 		(at 262.7715 726.4531 0)
 		(fields_autoplaced yes)
@@
 		)
 	)
-	(label "DH4"
+	(label "SH4"
 		(at 262.5131 695.1938 0)
 		(fields_autoplaced yes)
