File: Schematics/myth.kicad_sch (KiCad schematic)
At the start: 134 parts, among them J1 Conn_01x08_Male, J10 Conn_01x04_Male, J11 Conn_02x01, J2 Conn_01x08_Male, J3 Conn_01x08_Male, J4 Conn_01x08_Male, J5 Conn_01x08_Male, J6 Conn_01x08_Male, J8 Conn_01x08_Male, J9 Conn_01x04_Male, U1 74AHC02, U10 74HC595, U11 74HC165, U12 74AHC08, U13 74HC238, U14 74HC238, U15 74HC238, U16 4002, U17 74HC32, U18 74AHC273, U19 74LS32, U2 74AHC273, U20 CD4532BE, U21 74AHC138, U22 74AHC04, U23 74AHC138, U24 74HC238, U25 74HC238, U26 74LS32, U27 4078, U28 74AHC244, U29 74AHC138, U3 74HC74, U30 74AHC138, U31 4075, U32 74AHC02, U33 74AHC138, U34 74HC238, U35 74AHC138, U36 74HC163, U37 74AHC574, U38 74HC238, U39 74HC32, U4 74AHC04, U40 74AHC04, U41 74AHC574, U42 74HC74, U43 74AHC273, U44 74HC283, U45 74HC283, U46 74AHC273, U47 74HC02, U48 74HC157, U49 74HC157, U5 74AHC04, U50 74AHC244, U51 74AHC04, U52 74AHC574, U53 74HC193, U54 74HC193, U55 74HC193, U56 74HC193, U58 74HC193, U59 74HC193, U6 74AHC08, U60 74AHC244, U61 74LS32, U62 4078, U63 74AHC244, U64 74LS21, U65 74AHC04, U66 74AHC273, U67 74HC157, U68 74HC157, U69 74HC157, U7 74HC00, U70 74HC157, U71 74LS257, U72 74LS257, U73 74AHC273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

Commit message: Rename A register to GI
Connections:
- net DMx renamed MDx
- net DMx_pre renamed MDx_pre
- net LMx renamed MLx
- net LMx_pre renamed MLx_pre
- net xA renamed xGI
- net xDM_pre renamed xMD_pre
- net xLM_pre renamed xML_pre
- net ~{DMacc} renamed ~{MDacc}
- net ~{DMx} renamed ~{MDx}
- net ~{LMacc} renamed ~{MLacc}
- net ~{LMx} renamed ~{MLx}
- net ~{xDM} renamed ~{xMD}
- net ~{xLM} renamed ~{xML}
Other:
- note added: "Jump while loop counter register I not zero (decrements I)"
- note added: "Remap ("scrounge") RR, II etc, and impracticable opcodes such as N-MD"
- note removed: "ADD i"
- note removed: "Jump while value register I not zero (decrements I)"
- note removed: "Remap ("scrounge") MM, RR, DD etc, and impracticable opcodes such as NM"
- moved on the sheet: U19C
Changed lines of the file:
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@@
 	(wire
 		(pts
+			(xy 718.4214 525.7329) (xy 720.9614 525.7329)
+		)
+		(stroke
+			(width 0)
+			(type default)
+		)
+	)
+	(wire
+		(pts
 			(xy 1008.5848 564.7764) (xy 1031.7563 564.7764)
 		)
@@
 		)
 	)
-	(text "ADD i"
-		(exclude_from_sim no)
-		(at 367.9676 304.5504 0)
-		(effects
-			(font
-				(size 1.27 1.27)
-			)
-			(justify left bottom)
-		)
-	)
 	(text "IB 3-5 are the\nimmediate offset\nfor GET-PUT\noperations"
 		(exclude_from_sim no)
@@
 		)
 	)
-	(text "Jump while value register I not zero\n(decrements I)"
+	(text "Jump while loop counter register I not zero\n(decrements I)"
 		(exclude_from_sim no)
 		(at 65.8996 179.5348 0)
@@
 		)
 	)
-	(text "Remap (\"scrounge\") MM, RR, DD etc,\nand impracticable opcodes such as NM"
+	(text "Remap (\"scrounge\") RR, II etc,\nand impracticable opcodes such as N-MD"
 		(exclude_from_sim no)
 		(at 219.7394 228.2457 0)
@@
 		)
 	)
-	(label "~{DMx}"
+	(label "~{MDx}"
 		(at 705.7307 273.4183 180)
 		(fields_autoplaced yes)
@@
 		)
 	)
-	(label "~{xDM}"
+	(label "~{xMD}"
 		(at 1123.5198 503.8164 0)
 		(fields_autoplaced yes)
@@
 		)
 	)
-	(label "~{LMacc}"
-		(at 733.6614 528.2729 0)
+	(label "~{MLacc}"
+		(at 736.2014 528.2729 0)
 		(fields_autoplaced yes)
 		(effects
@@
 		)
 	)
-	(label "~{DMacc}"
+	(label "~{MDacc}"
 		(at 973.2338 692.6042 0)
 		(fields_autoplaced yes)
@@
 		)
 	)
-	(label "xA"
+	(label "xGI"
 		(at 364.9218 304.4698 0)
 		(fields_autoplaced yes)
@@
 		)
 	)
-	(label "~{xLM}"
+	(label "~{xML}"
 		(at 364.2868 268.9098 0)
 		(fields_autoplaced yes)
@@
 		)
 	)
-	(label "DMx_pre"
+	(label "MDx_pre"
 		(at 137.3886 380.1872 0)
 		(fields_autoplaced yes)
@@
 		)
 	)
-	(label "LMx"
+	(label "MLx"
 		(at 759.5384 199.9363 0)
 		(fields_autoplaced yes)
@@
 		)
 	)
-	(label "~{xLM}"
+	(label "~{xML}"
 		(at 1123.5198 506.3564 0)
 		(fields_autoplaced yes)
@@
 		)
 	)
-	(label "xDM_pre"
+	(label "xMD_pre"
 		(at 957.9938 695.1442 180)
 		(fields_autoplaced yes)
@@
 		)
 	)
-	(label "~{LMacc}"
+	(label "~{MLacc}"
 		(at 666.674 517.1937 180)
 		(fields_autoplaced yes)
@@
 		)
 	)
-	(label "LMx_pre"
+	(label "MLx_pre"
 		(at 137.3886 382.7272 0)
 		(fields_autoplaced yes)
@@
 		)
 	)
-	(label "DMx_pre"
+	(label "MDx_pre"
 		(at 957.9938 690.0642 180)
 		(fields_autoplaced yes)
@@
 		)
 	)
-	(label "xA"
+	(label "xGI"
 		(at 594.1685 186.1343 180)
 		(fields_autoplaced yes)
@@
 		)
 	)
-	(label "LMx_pre"
+	(label "MLx_pre"
 		(at 703.1814 523.1929 180)
 		(fields_autoplaced yes)
@@
 		)
 	)
-	(label "xA"
+	(label "xGI"
 		(at 562.7742 167.7322 180)
 		(fields_autoplaced yes)
@@
 		)
 	)
-	(label "DMx"
+	(label "MDx"
 		(at 720.9707 273.4183 0)
 		(fields_autoplaced yes)
@@
 		)
 	)
-	(label "xLM_pre"
+	(label "xML_pre"
 		(at 175.1584 279.1714 180)
 		(fields_autoplaced yes)
@@
 		)
 	)
-	(label "~{DMx}"
+	(label "~{MDx}"
 		(at 362.3818 376.2248 0)
 		(fields_autoplaced yes)
@@
 		)
 	)
-	(label "~{xDM}"
+	(label "~{xMD}"
 		(at 364.2868 266.3698 0)
 		(fields_autoplaced yes)
@@
 		)
 	)
-	(label "xLM_pre"
+	(label "xML_pre"
 		(at 131.1148 316.5348 0)
 		(fields_autoplaced yes)
@@
 		)
 	)
-	(label "~{DMacc}"
+	(label "~{MDacc}"
 		(at 948.6797 657.1799 180)
 		(fields_autoplaced yes)
@@
 		)
 	)
-	(label "~{LMx}"
+	(label "~{MLx}"
 		(at 744.2984 199.9363 180)
 		(fields_autoplaced yes)
@@
 		)
 	)
-	(label "LMx"
+	(label "MLx"
 		(at 1109.2883 604.7814 0)
 		(fields_autoplaced yes)
@@
 	)
 	(label "GETPUT"
-		(at 718.4214 530.8129 180)
+		(at 720.9614 530.8129 180)
 		(fields_autoplaced yes)
 		(effects
@@
 		)
 	)
-	(label "xDM_pre"
+	(label "xMD_pre"
 		(at 131.1148 313.9948 0)
 		(fields_autoplaced yes)
@@
 		)
 	)
-	(label "DMx_pre"
+	(label "MDx_pre"
 		(at 174.9866 261.5757 180)
 		(fields_autoplaced yes)
@@
 		)
 	)
-	(label "DMx"
+	(label "MDx"
 		(at 1109.2883 602.2414 0)
 		(fields_autoplaced yes)
@@
 		)
 	)
-	(label "xDM_pre"
+	(label "xMD_pre"
 		(at 175.1584 284.2514 180)
 		(fields_autoplaced yes)
@@
 		)
 	)
-	(label "xA"
+	(label "xGI"
 		(at 562.9238 225.3634 180)
 		(fields_autoplaced yes)
@@
 		)
 	)
-	(label "LMx_pre"
+	(label "MLx_pre"
 		(at 174.9866 256.4957 180)
 		(fields_autoplaced yes)
@@
 		)
 	)
-	(label "~{LMx}"
+	(label "~{MLx}"
 		(at 362.3818 378.7648 0)
 		(fields_autoplaced yes)
@@
 		)
 	)
-	(label "xLM_pre"
+	(label "xML_pre"
 		(at 703.1814 528.2729 180)
 		(fields_autoplaced yes)
@@
 	(symbol
 		(lib_id "74xx:74LS32")
-		(at 726.0414 528.2729 0)
+		(at 728.5814 528.2729 0)
 		(unit 3)
 		(exclude_from_sim no)
@@
 		(fields_autoplaced yes)
 		(property "Reference" "U19"
-			(at 726.0414 520.3184 0)
+			(at 728.5814 520.3184 0)
 			(effects
 				(font
@@
 		)
 		(property "Value" "74LS32"
-			(at 726.0414 522.7427 0)
+			(at 728.5814 522.7427 0)
 			(effects
 				(font
@@
 		)
 		(property "Footprint" ""
-			(at 726.0414 528.2729 0)
+			(at 728.5814 528.2729 0)
 			(effects
 				(font
@@
 		)
 		(property "Datasheet" "http://www.ti.com/lit/gpn/sn74LS32"
-			(at 726.0414 528.2729 0)
+			(at 728.5814 528.2729 0)
 			(effects
 				(font
@@
 		)
 		(property "Description" "Quad 2-input OR"
-			(at 726.0414 528.2729 0)
+			(at 728.5814 528.2729 0)
 			(effects
 				(font

Commit message: Rename WTF to JW, JT, JF for clarity
Connections:
- net xF renamed xJF
- net xT renamed xJT
- net xW renamed xJW
- net xW_pre renamed xJW_pre
- net ~{xW} renamed ~{xJW}
Changed lines of the file:
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@@
 		)
 	)
-	(label "xT"
+	(label "xJT"
 		(at 63.9318 196.3674 180)
 		(fields_autoplaced yes)
@@
 		)
 	)
-	(label "xW"
+	(label "xJW"
 		(at 745.0077 134.3281 180)
 		(fields_autoplaced yes)
@@
 		)
 	)
-	(label "xW_pre"
+	(label "xJW_pre"
 		(at 63.9318 191.2874 180)
 		(fields_autoplaced yes)
@@
 		)
 	)
-	(label "~{xW}"
+	(label "~{xJW}"
 		(at 760.2477 134.3281 0)
 		(fields_autoplaced yes)
@@
 		)
 	)
-	(label "xW_pre"
+	(label "xJW_pre"
 		(at 131.6482 269.5702 0)
 		(fields_autoplaced yes)
@@
 		)
 	)
-	(label "xT"
+	(label "xJT"
 		(at 364.9218 314.6298 0)
 		(fields_autoplaced yes)
@@
 		)
 	)
-	(label "xF"
+	(label "xJF"
 		(at 364.9218 317.1698 0)
 		(fields_autoplaced yes)
@@
 		)
 	)
-	(label "~{xW}"
+	(label "~{xJW}"
 		(at 631.5591 667.5672 180)
 		(fields_autoplaced yes)
@@
 		)
 	)
-	(label "xW"
+	(label "xJW"
 		(at 364.9218 312.0898 0)
 		(fields_autoplaced yes)
@@
 		)
 	)
-	(label "xF"
+	(label "xJF"
 		(at 63.9318 198.9074 180)
 		(fields_autoplaced yes)

Commit message: Add INO/DEO scrounge opcodes
Parts:
- removed U74: 74AHC273, Package_DIP:DIP-20_W7.62mm_Socket_LongPads, symbol 74xx:74HC273
- added U57, U95: 74HC193, Package_DIP:DIP-16_W7.62mm_Socket_LongPads, symbol 74xx:74LS193
Connections:
- net +5V: now also U57.16 (VCC), U95.16 (VCC)
- net GND: now also U39.10, U39.9, U57.8 (GND), U95.8 (GND); no longer U1.8, U1.9, U7.1, U7.2
- net O0: now also U57.3 (QA)
- net O1: now also U57.2 (QB)
- net O2: now also U57.6 (QC)
- net O3: now also U57.7 (QD)
- net O4: now also U95.3 (QA)
- net O5: now also U95.2 (QB)
- net O6: now also U95.6 (QC)
- net O7: now also U95.7 (QD)
- net RES: now also U57.14 (CLR), U95.14 (CLR)
- net INO: now reaches U27.2, U6.6
- net INO: now also U7.1, U7.2
- net at U17.3: now also U1.9; no longer U39.10
- net at U39.11, U69.1 (S), U70.1 (S): now also U1.8; no longer U39.9
- net at U1.10: now also U57.11 (~{LOAD}), U95.11 (~{LOAD})
- net DEO: now reaches U22.13, U27.3, U6.3
- net ~{DEO}: now reaches U22.12, U8.12
- net ~{DEO}: now also U57.4 (DOWN)
- net at U70.12 (Zd): now also U57.9 (D)
- net at U70.4 (Za): now also U57.15 (A)
- net at U70.7 (Zb): now also U57.1 (B)
- net at U70.9 (Zc): now also U57.10 (C)
- net at U69.12 (Zd): now also U95.9 (D)
- net at U69.4 (Za): now also U95.15 (A)
- net at U69.7 (Zb): now also U95.1 (B)
- net at U69.9 (Zc): now also U95.10 (C)
- net ~{INO}: now reaches U7.3
- net ~{INO}: now also U57.5 (UP)
- new net ~{BOO}: U57.13 (~{BO}), U95.4 (DOWN)
- new net ~{COO}: U57.12 (~{CO}), U95.5 (UP)
- no-connect marks 65 -> 66
Other:
- note added: "Most mapped to NOP, but reserved for instruction set extensions"
- note added: "To do: Fix logic above to map NML to INO, and NMD to DEO"
- note removed: "Currently mapped to NOP, reserved for instruction set extensions"
- note removed: "O provides the return offset during RET receives the return offset during SUBR can be GET and PUT provides all address offsets except FETCH can be stored into is the implied 2nd ALU input operand"
- moved on the sheet: U17A, U1C, U39C, U39D, U69, U70, U79, U7A
