File: Schematics/myth_cdl/dreg.kicad_sch (KiCad schematic)
At the start: 6 parts, among them U15 74HC193, U16 74HC193, U17 74AHC244, U18 74AHC574, U5 74LS08, U7 74HC02

Commit message: Change d to g
Parts:
- U5, U7: footprint (none) -> Package_DIP:DIP-14_W7.62mm_LongPads
Changed lines of the file:
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@@
 			)
 		)
-		(property "Footprint" ""
+		(property "Footprint" "Package_DIP:DIP-14_W7.62mm_LongPads"
 			(at 153.67 105.41 0)
 			(effects
@@
 			)
 		)
-		(property "Footprint" ""
+		(property "Footprint" "Package_DIP:DIP-14_W7.62mm_LongPads"
 			(at 49.53 125.73 0)
 			(effects
@@
 			)
 		)
-		(property "Footprint" ""
+		(property "Footprint" "Package_DIP:DIP-14_W7.62mm_LongPads"
 			(at 201.93 86.36 0)
 			(effects
@@
 			)
 		)
-		(property "Footprint" ""
+		(property "Footprint" "Package_DIP:DIP-14_W7.62mm_LongPads"
 			(at 173.99 107.95 0)
 			(effects
