File: Schematics/myth_decoder/sys_trap_getput.kicad_sch (KiCad schematic)
At the start: 7 parts, among them U13 74AHC04, U19 74HC02, U2 74LS08, U20 74AHC138, U21 74AHC138, U22 74AHC244, U3 74LS32

Commit message: Change d to g
Parts:
- added C1013: C 100nF, Capacitor_THT:C_Disc_D5.0mm_W2.5mm_P2.50mm, symbol Device:C_Small
- added C1014: CP 10μF, Capacitor_THT:CP_Radial_D6.3mm_P2.50mm, symbol Device:C_Polarized_Small
- renumbered U2 to U1002, U3 to U1003, U13 to U1013, U19 to U1019, U20 to U1020, U21 to U1021, U22 to U1022
Connections:
- net +5V: now also C1013.1, C1014.1
- net GND: now also C1013.2, C1014.2
