File: Schematics/myth_io/enable.kicad_sch (KiCad schematic)
At the start: 5 parts, among them U11 74AHC273, U12 74HC238, U13 74HC238, U14 74AHC138, U15 74AHC138

Commit message: Change CO do D
Parts:
- removed U14, U15: 74AHC138, Package_DIP:DIP-16_W7.62mm_Socket_LongPads, symbol 74xx:74LS138
- added U1014, U1015: 74HC238, Package_DIP:DIP-16_W7.62mm_Socket_LongPads, symbol 74xx:74HC238
- renumbered U11 to U1011, U12 to U1012, U13 to U1013
Connections:
- net +5V: now also U1014.16 (VCC), U1014.6 (E3), U1015.16 (VCC)
- net EL0: now also U1014.1 (A0), U1015.1 (A0)
- net EL1: now also U1014.2 (A1), U1015.2 (A1)
- net EL2: now also U1014.3 (A2), U1015.3 (A2)
- net EL3: now also U1014.4 (~{E1}), U1015.6 (E3)
- net GND: now also U1014.5 (~{E2}), U1014.8 (GND), U1015.4 (~{E1}), U1015.5 (~{E2}), U1015.8 (GND)
- new net SL0_NULL: U1014.15 (Y0)
- new net SL10: U1015.13 (Y2)
- new net SL11: U1015.12 (Y3)
- new net SL12: U1015.11 (Y4)
- new net SL13: U1015.10 (Y5)
- new net SL14: U1015.9 (Y6)
- new net SL15: U1015.7 (Y7)
- new net SL1_PAROE: U1014.14 (Y1)
- new net SL2: U1014.13 (Y2)
- new net SL3: U1014.12 (Y3)
- new net SL4: U1014.11 (Y4)
- new net SL5: U1014.10 (Y5)
- new net SL6: U1014.9 (Y6)
- new net SL7: U1014.7 (Y7)
- new net SL8: U1015.15 (Y0)
- new net SL9: U1015.14 (Y1)
Other:
- note added: "HIGH ORDER SELECTOR"
- note added: "LOW ORDER SELECTOR"
- note removed: "ACTIVE HIGH ENABLE"
- note removed: "ACTIVE LOW ENABLE"
