File: Schematics/myth_io/parallel.kicad_sch (KiCad schematic)
At the start: 4 parts, among them U10 74AHC574, U5 74AHC04, U9 74AHC574

Commit message: Change CO do D
Parts:
- added unit 5 of U1003
- renumbered RN2 to RN1002, U5 to U1003, U9 to U1009, U10 to U1010
Connections:
- net ~{SL1_PAROE}: no longer names the net of U1009.1 (OE)
- net ~{SL1_PAROE}: now also U1003.10
- new net SL1_PAROE: U1003.11
Changed lines of the file:
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@@
+	(wire
+		(pts
+			(xy 81.28 121.92) (xy 92.71 121.92)
+		)
+		(stroke
+			(width 0)
+			(type default)
+		)
+	)
 	(wire
 		(pts
@@
 		)
 	)
-	(global_label "~{SL1_PAROE}"
+	(global_label "SL1_PAROE"
 		(shape input)
-		(at 92.71 121.92 180)
+		(at 66.04 121.92 180)
 		(fields_autoplaced yes)
 		(effects
@@
 		)
 		(property "Intersheetrefs" "${INTERSHEET_REFS}"
-			(at 79.202 121.92 0)
+			(at 52.532 121.92 0)
 			(effects
 				(font
@@
 		(on_board yes)
 		(dnp no)
-		(property "Reference" "RN2"
+		(property "Reference" "RN1002"
 			(at 109.22 139.065 90)
 			(effects
@@
 			(project "myth_io"
 				(path "/a907dd88-e0e4-4e6e-a291-053f6213a316/afcac29e-dbf8-41a5-a4eb-0c249df1dff5"
-					(reference "RN2")
+					(reference "RN1002")
 					(unit 1)
 				)
@@
 		(dnp no)
 		(fields_autoplaced yes)
-		(property "Reference" "U5"
+		(property "Reference" "U1003"
 			(at 154.94 82.55 0)
 			(effects
@@
 			(project "myth_io"
 				(path "/a907dd88-e0e4-4e6e-a291-053f6213a316/afcac29e-dbf8-41a5-a4eb-0c249df1dff5"
-					(reference "U5")
+					(reference "U1003")
 					(unit 4)
 				)
@@
 		(on_board yes)
 		(dnp no)
-		(property "Reference" "U9"
+		(property "Reference" "U1009"
 			(at 105.41 84.3026 0)
 			(effects
@@
 			(project "myth_io"
 				(path "/a907dd88-e0e4-4e6e-a291-053f6213a316/afcac29e-dbf8-41a5-a4eb-0c249df1dff5"
-					(reference "U9")
+					(reference "U1009")
 					(unit 1)
+				)
+			)
+		)
+	)
+	(symbol
+		(lib_id "74xx:74AHC04")
+		(at 73.66 121.92 0)
+		(unit 5)
+		(exclude_from_sim no)
+		(in_bom yes)
+		(on_board yes)
+		(dnp no)
+		(fields_autoplaced yes)
+		(property "Reference" "U1003"
+			(at 73.66 113.03 0)
+			(effects
+				(font
+					(size 1.27 1.27)
+				)
+			)
+		)
+		(property "Value" "74AHC04"
+			(at 73.66 115.57 0)
+			(effects
+				(font
+					(size 1.27 1.27)
+				)
+			)
+		)
+		(property "Footprint" "Package_DIP:DIP-14_W7.62mm_Socket_LongPads"
+			(at 73.66 121.92 0)
+			(effects
+				(font
+					(size 1.27 1.27)
+				)
+				(hide yes)
+			)
+		)
+		(property "Datasheet" "https://assets.nexperia.com/documents/data-sheet/74AHC_AHCT04.pdf"
+			(at 73.66 121.92 0)
+			(effects
+				(font
+					(size 1.27 1.27)
+				)
+				(hide yes)
+			)
+		)
+		(property "Description" "Hex Inverter"
+			(at 73.66 121.92 0)
+			(effects
+				(font
+					(size 1.27 1.27)
+				)
+				(hide yes)
+			)
+		)
+		(pin "6"
+		)
+		(pin "13"
+		)
+		(pin "14"
+		)
+		(pin "7"
+		)
+		(pin "12"
+		)
+		(pin "1"
+		)
+		(pin "10"
+		)
+		(pin "11"
+		)
+		(pin "5"
+		)
+		(pin "4"
+		)
+		(pin "8"
+		)
+		(pin "2"
+		)
+		(pin "3"
+		)
+		(pin "9"
+		)
+		(instances
+			(project "myth_io"
+				(path "/a907dd88-e0e4-4e6e-a291-053f6213a316/afcac29e-dbf8-41a5-a4eb-0c249df1dff5"
+					(reference "U1003")
+					(unit 5)
 				)
 			)
@@
 		(on_board yes)
 		(dnp no)
-		(property "Reference" "U10"
+		(property "Reference" "U1010"
 			(at 168.91 32.2326 0)
 			(effects
@@
 			(project "myth_io"
 				(path "/a907dd88-e0e4-4e6e-a291-053f6213a316/afcac29e-dbf8-41a5-a4eb-0c249df1dff5"
-					(reference "U10")
+					(reference "U1010")
 					(unit 1)
 				)
