File: Schematics/old/myth.kicad_sch (KiCad schematic)
At the start: 140 parts, among them J1 Conn_01x08_Male, J10 Conn_02x01, J2 Conn_01x08_Male, J3 Conn_01x08_Male, J4 Conn_01x08_Male, J5 Conn_01x08_Male, J6 Conn_01x08_Male, J7 Conn_01x08_Male, J8 Conn_01x04_Male, J9 Conn_01x04_Male, U1 74AHC02, U10 74HC595, U11 74HC165, U12 74AHC08, U13 74HC238, U14 74HC238, U15 74HC238, U16 4002, U17 74AHC273, U18 74LS32, U19 CD4532BE, U2 74AHC04, U20 74AHC138, U21 74AHC04, U22 74AHC138, U23 74HC238, U24 74HC238, U25 74LS32, U26 4078, U27 74AHC244, U28 74LS08, U29 74HC238, U3 74HC74, U30 74HC238, U31 4075, U32 74AHC04, U33 74HC00, U34 74HC163, U35 74AHC138, U36 74AHC138, U37 74HC238, U38 74AHC138, U39 74HC238, U4 74HC32, U40 74AHC02, U41 74AHC574, U42 74HC283, U43 74HC283, U44 74AHC574, U45 74HC193, U46 74HC193, U47 74HC157, U48 74HC157, U49 74HC32, U5 74AHC273, U50 74AHC244, U51 74HC157, U52 74HC157, U53 74HC157, U54 74HC157, U55 74HC02, U56 74HC74, U57 74HC193, U58 74HC193, U59 74HC04, U6 74LS08, U60 4078, U61 4078, U62 74AHC574, U63 74HC193, U64 74HC193, U65 74AHC273, U66 74AHC273, U67 74LS573, U68 74LS21, U69 74AHC244, U7 74AHC08, U70 74AHC04, U71 74AHC04, U72 74LS32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

Commit message: Fix documentation re: change d->g
Parts:
- added C25: C_Small, Capacitor_THT:C_Disc_D5.0mm_W2.5mm_P2.50mm, symbol Device:C_Small
Connections:
- net EHL is gone; now on net EL3: U29.4 (~{G2A})
- net GND: now also C25.1
- net at J2.2 (Pin_2), R2.2, U2.5: now also C25.2
Other:
- note added: "FREE signals that code execution is outside the TRAP region (pages 0-31): Intererrupts are disabled when executing within pages 0-31."
- note removed: "FREE signals that code execution is outside the TRAP region (pages 0-31): Intererrupts are enabled, iff this is the case"
- moved on the sheet: R2
Changed lines of the file:
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@@
 	)
 	(junction
+		(at 85.09 95.25)
+		(diameter 0)
+		(color 0 0 0 0)
+	)
+	(junction
 		(at 394.97 668.02)
 		(diameter 0)
@@
 	)
 	(junction
-		(at 85.09 95.25)
-		(diameter 0)
-		(color 0 0 0 0)
-	)
-	(junction
 		(at 703.58 778.51)
 		(diameter 0)
@@
 	(wire
 		(pts
-			(xy 85.09 107.95) (xy 83.82 107.95)
+			(xy 85.09 76.2) (xy 83.82 76.2)
 		)
 		(stroke
@@
 	(wire
 		(pts
-			(xy 71.12 107.95) (xy 76.2 107.95)
+			(xy 71.12 76.2) (xy 76.2 76.2)
 		)
 		(stroke
@@
 	(wire
 		(pts
+			(xy 85.09 95.25) (xy 100.33 95.25)
+		)
+		(stroke
+			(width 0)
+			(type default)
+		)
+	)
+	(wire
+		(pts
 			(xy 311.15 279.4) (xy 311.15 306.07)
 		)
@@
 	(wire
 		(pts
-			(xy 85.09 95.25) (xy 100.33 95.25)
+			(xy 82.55 95.25) (xy 85.09 95.25)
 		)
 		(stroke
@@
 	(wire
 		(pts
+			(xy 85.09 114.3) (xy 85.09 120.65)
+		)
+		(stroke
+			(width 0)
+			(type default)
+		)
+	)
+	(wire
+		(pts
 			(xy 425.45 553.72) (xy 425.45 556.26)
 		)
@@
 	(wire
 		(pts
+			(xy 85.09 76.2) (xy 85.09 95.25)
+		)
+		(stroke
+			(width 0)
+			(type default)
+		)
+	)
+	(wire
+		(pts
 			(xy 90.17 678.18) (xy 90.17 685.8)
 		)
@@
 	(wire
 		(pts
+			(xy 85.09 95.25) (xy 85.09 109.22)
+		)
+		(stroke
+			(width 0)
+			(type default)
+		)
+	)
+	(wire
+		(pts
 			(xy 998.22 170.18) (xy 998.22 172.72)
 		)
@@
 	(wire
 		(pts
-			(xy 82.55 95.25) (xy 85.09 95.25)
-		)
-		(stroke
-			(width 0)
-			(type default)
-		)
-	)
-	(wire
-		(pts
 			(xy 582.93 148.59) (xy 605.79 148.59)
 		)
@@
 		)
 	)
-	(wire
-		(pts
-			(xy 85.09 107.95) (xy 85.09 95.25)
-		)
-		(stroke
-			(width 0)
-			(type default)
-		)
-	)
 	(polyline
 		(pts
@@
 		)
 	)
-	(text "FREE signals that\ncode execution is\noutside the TRAP\nregion (pages 0-31):\nIntererrupts are\nenabled, iff\nthis is the case\n"
+	(text "FREE signals that\ncode execution is\noutside the TRAP\nregion (pages 0-31):\nIntererrupts are\ndisabled when\nexecuting within\npages 0-31."
 		(exclude_from_sim no)
-		(at 43.18 491.49 0)
+		(at 43.18 493.522 0)
 		(effects
 			(font
@@
 	(text "~{RES} request"
 		(exclude_from_sim no)
-		(at 73.66 88.9 0)
+		(at 67.056 88.392 0)
 		(effects
 			(font
@@
 		)
 	)
-	(label "EHL"
+	(label "EL3"
 		(at 280.67 669.29 180)
 		(fields_autoplaced yes)
@@
 	)
 	(label "+5V"
-		(at 71.12 107.95 180)
+		(at 71.12 76.2 180)
 		(fields_autoplaced yes)
 		(effects
@@
 	(symbol
 		(lib_id "Device:R")
-		(at 80.01 107.95 90)
+		(at 80.01 76.2 90)
 		(unit 1)
 		(exclude_from_sim no)
@@
 		(dnp no)
 		(property "Reference" "R2"
-			(at 80.01 113.2078 90)
+			(at 80.01 81.4578 90)
 			(effects
 				(font
@@
 		)
 		(property "Value" "R7.5k"
-			(at 80.01 110.8964 90)
+			(at 80.01 79.1464 90)
 			(effects
 				(font
@@
 		)
 		(property "Footprint" "Resistor_THT:R_Axial_DIN0207_L6.3mm_D2.5mm_P10.16mm_Horizontal"
-			(at 80.01 109.728 90)
+			(at 80.01 77.978 90)
 			(effects
 				(font
@@
 		)
 		(property "Datasheet" "~"
-			(at 80.01 107.95 0)
+			(at 80.01 76.2 0)
 			(effects
 				(font
@@
 		)
 		(property "Description" ""
-			(at 80.01 107.95 0)
+			(at 80.01 76.2 0)
 			(effects
 				(font
@@
 	)
 	(symbol
+		(lib_id "power:GND")
+		(at 85.09 120.65 0)
+		(unit 1)
+		(exclude_from_sim no)
+		(in_bom yes)
+		(on_board yes)
+		(dnp no)
+		(property "Reference" "#PWR036"
+			(at 85.09 127 0)
+			(effects
+				(font
+					(size 1.27 1.27)
+				)
+				(hide yes)
+			)
+		)
+		(property "Value" "GND"
+			(at 85.217 125.0442 0)
+			(effects
+				(font
+					(size 1.27 1.27)
+				)
+			)
+		)
+		(property "Footprint" ""
+			(at 85.09 120.65 0)
+			(effects
+				(font
+					(size 1.27 1.27)
+				)
+				(hide yes)
+			)
+		)
+		(property "Datasheet" ""
+			(at 85.09 120.65 0)
+			(effects
+				(font
+					(size 1.27 1.27)
+				)
+				(hide yes)
+			)
+		)
+		(property "Description" ""
+			(at 85.09 120.65 0)
+			(effects
+				(font
+					(size 1.27 1.27)
+				)
+				(hide yes)
+			)
+		)
+		(pin "1"
+		)
+		(instances
+			(project "myth"
+				(path "/29cbb0bc-f66b-4d11-80e7-5bb270e42496"
+					(reference "#PWR036")
+					(unit 1)
+				)
+			)
+		)
+	)
+	(symbol
 		(lib_id "74xx:74HC04")
 		(at 708.66 203.2 0)
@@
 					(unit 1)
 				)
+			)
+		)
+	)
+	(symbol
+		(lib_id "Device:C_Small")
+		(at 85.09 111.76 180)
+		(unit 1)
+		(exclude_from_sim no)
+		(in_bom yes)
+		(on_board yes)
+		(dnp no)
+		(property "Reference" "C25"
+			(at 82.7532 112.9284 0)
+			(effects
+				(font
+					(size 1.27 1.27)
+				)
+				(justify left)
+			)
+		)
+		(property "Value" "C_Small"
+			(at 82.7532 110.617 0)
+			(effects
+				(font
+					(size 1.27 1.27)
+				)
+				(justify left)
+			)
+		)
+		(property "Footprint" "Capacitor_THT:C_Disc_D5.0mm_W2.5mm_P2.50mm"
+			(at 85.09 111.76 0)
+			(effects
+				(font
+					(size 1.27 1.27)
+				)
+				(hide yes)
+			)
+		)
+		(property "Datasheet" "~"
+			(at 85.09 111.76 0)
+			(effects
+				(font
+					(size 1.27 1.27)
+				)
+				(hide yes)
+			)
+		)
+		(property "Description" ""
+			(at 85.09 111.76 0)
+			(effects
+				(font
+					(size 1.27 1.27)
+				)
+				(hide yes)
+			)
+		)
+		(pin "1"
+		)
+		(pin "2"
+		)
+		(instances
+			(project "myth"
+				(path "/29cbb0bc-f66b-4d11-80e7-5bb270e42496"
+					(reference "C25")
+					(unit 1)
+				)

Commit message: Change semantics of xB
Parts:
- removed U47, U48: 74HC157, Package_DIP:DIP-16_W7.62mm_Socket_LongPads, symbol 74xx:74LS157
- added U47: 74AHC273, Package_DIP:DIP-20_W7.62mm_Socket_LongPads, symbol 74xx:74HC273
Connections:
- net +5V: now also U47.20 (VCC); no longer U45.11 (~{LOAD}), U46.11 (~{LOAD})
- net CLOSE: now also U47.11 (Cp)
- net DB0: now also U53.3 (I1a)
- net DB1: now also U53.6 (I1b)
- net DB2: now also U53.10 (I1c)
- net DB3: now also U53.13 (I1d)
- net DB4: now also U54.3 (I1a)
- net DB5: now also U54.6 (I1b)
- net DB6: now also U54.10 (I1c)
- net DB7: now also U54.13 (I1d)
- net GND: now also U6.4, U6.5, U47.10 (GND); no longer U2.9, U45.1 (B), U45.10 (C), U45.15 (A), U45.9 (D), U46.1 (B), U46.10 (C), U46.15 (A), U46.9 (D)
- net I0: no longer U42.6 (B1)
- net I1: no longer U42.2 (B2)
- net I2: no longer U42.15 (B3)
- net I3: no longer U42.11 (B4)
- net I4: no longer U43.6 (B1)
- net I5: no longer U43.2 (B2)
- net I6: no longer U43.15 (B3)
- net I7: no longer U43.11 (B4)
- net JUMP: now also U33.12; no longer U6.5
- net ~{RES}: now also U47.1 (~{Mr})
- net ~{xLFIX}: now reaches U2.8
- net ~{xLFIX}: now also U45.11 (~{LOAD}), U46.11 (~{LOAD})
- net at U6.6: no longer U33.12
- net at U42.1 (S2): now also U45.1 (B)
- net at U42.10 (S4): now also U45.9 (D)
- net at U42.13 (S3): now also U45.10 (C)
- net at U42.4 (S1): now also U45.15 (A)
- net at U45.2 (QB), U50.4 (1A1): now also U47.4 (D1)
- net at U45.3 (QA), U50.2 (1A0): now also U47.3 (D0)
- net at U45.6 (QC), U50.6 (1A2): now also U47.7 (D2)
- net at U45.7 (QD), U50.8 (1A3): now also U47.8 (D3)
- net at U43.1 (S2): now also U46.1 (B)
- net at U43.10 (S4): now also U46.9 (D)
- net at U43.13 (S3): now also U46.10 (C)
- net at U43.4 (S1): now also U46.15 (A)
- net at U46.7 (QD), U50.11 (2A3): now also U47.18 (D7)
- net at U46.6 (QC), U50.13 (2A2): now also U47.17 (D6)
- net at U46.2 (QB), U50.15 (2A1): now also U47.14 (D5)
- net at U46.3 (QA), U50.17 (2A0): now also U47.13 (D4)
- net Lx renamed MLx
- net Lx_pre renamed MLx_pre
- net Mx renamed MGx
- net Mx_pre renamed MGx_pre
- net opc_FIX renamed opc_RFIX
- net xB renamed xLFIX
- net xLFIX: now also U2.9; no longer U6.4
- net xL_pre renamed xML_pre
- net xM_pre renamed xMG_pre
- net ~{Lx} renamed ~{MLx}
- net ~{Mx} renamed ~{MGx}
- net ~{opc_FIX} renamed ~{opc_RFIX}
- net ~{xL} renamed ~{xML}
- net ~{xM} renamed ~{xMG}
- new net L0: U42.6 (B1), U47.2 (Q0)
- new net L1: U42.2 (B2), U47.5 (Q1)
- new net L2: U42.15 (B3), U47.6 (Q2)
- new net L3: U42.11 (B4), U47.9 (Q3)
- new net L4: U43.6 (B1), U47.12 (Q4)
- new net L5: U43.2 (B2), U47.15 (Q5)
- new net L6: U43.15 (B3), U47.16 (Q6)
- new net L7: U43.11 (B4), U47.19 (Q7)
Other:
- note added: "(Coroutine Latch)"
- note added: "ALT: COxML7"
- note added: "CO"
- note added: "Instruction byte: all0: OPC_SYS 00000 xxx See table @ SYS decoder else: opc_RFIX 00001 x xx b0-1 LSB, b2: Extended sign bit OPC_ALU 0001 xxxx See table @ ALU OPC_TRAP 001 xxxxx b0-4: DEST PAGE OPC_GIRO 01 xx x xxx b0-2 OFFS, b3:GET/PUT, B4-5:REG(GIRO) OPC_PAIR 1 xxx xxxx b0-3 DST, b4-6 SRC"
- note added: "MGx"
- note added: "xMG"
- note removed: "(DUPE) Register"
- note removed: "ALT: COxL7"
- note removed: "D"
- note removed: "Instruction byte: all0: OPC_SYS 00000 xxx See table @ SYS decoder else: OPC_FIX 00001 x xx b0-1 LSB, b2: Extended sign bit OPC_ALU 0001 xxxx See table @ ALU OPC_TRAP 001 xxxxx b0-4: DEST PAGE OPC_GIRO 01 xx x xxx b0-2 OFFS, b3:GET/PUT, B4-5:REG(GIRO) OPC_PAIR 1 xxx xxxx b0-3 DST, b4-6 SRC"
- note removed: "Mx"
- note removed: "Relative Addressing"
- note removed: "xM"
- moved on the sheet: U18C, U1C, U28B, U32B, U32C, U32E, U33D, U40A, U4A, U50, U56B, U59B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

Commit message: Change signal names
Connections:
- net Nx renamed FETCHx
- net Nx_pre renamed FETCHx_pre
- net Nx_pre_clean renamed FETCHx_pre_clean
- net xA renamed xSKIP
- net xC renamed xCALL
- net xF renamed xJRF
- net xJ renamed xJMP
- net xT renamed xJRT
- net xW renamed xJWIT
- net xW_pre renamed xJWIT_pre
- net ~{Nx} renamed ~{FETCHx}
- net ~{xW} renamed ~{xJWIT}
Other:
- note added: "8 AND (R:=R&O) 9 IOR (R:=R|O) 10 EOR (R:=R^O) 11 ADD (Add" / R:=R+O, bits 0-7) 12 CAR ("Carry Bit" / R:= Carry, 9th bit of R+O) 00h or 01h 13 RLO ("Flag: R less than O" / R:= (R<O)? 0xJRFF:0 14 REO ("Flag: R equals O" / R:= (R==O)? 0xJRFF:0 15 RGO ("Flag: R greater than O" / R:= (R>O)? 0xJRFF:0"
- note added: "Else sign exJRTend bit 2"
- note added: "Instruction byte: all0: OPC_SYS 00000 xxx See table @ SYS decoder else: opc_RFIX 00001 x xx b0-1 LSB, b2: ExJRTended sign bit OPC_ALU 0001 xxxx See table @ ALU OPC_TRAP 001 xxxxx b0-4: DEST PAGE OPC_GIRO 01 xx x xxx b0-2 OFFS, b3:GET/PUT, B4-5:REG(GIRO) OPC_PAIR 1 xxx xxxx b0-3 DST, b4-6 SRC"
- note added: "Mapped to NOP, but reserved for instruction set exJRTensions"
- note added: "xSKIP adds DB val to O and carries over into D"
- note removed: "8 AND (R:=R&O) 9 IOR (R:=R|O) 10 EOR (R:=R^O) 11 ADD (Add" / R:=R+O, bits 0-7) 12 CAR ("Carry Bit" / R:= Carry, 9th bit of R+O) 00h or 01h 13 RLO ("Flag: R less than O" / R:= (R<O)? 0xFF:0 14 REO ("Flag: R equals O" / R:= (R==O)? 0xFF:0 15 RGO ("Flag: R greater than O" / R:= (R>O)? 0xFF:0"
- note removed: "Else sign extend bit 2"
- note removed: "Instruction byte: all0: OPC_SYS 00000 xxx See table @ SYS decoder else: opc_RFIX 00001 x xx b0-1 LSB, b2: Extended sign bit OPC_ALU 0001 xxxx See table @ ALU OPC_TRAP 001 xxxxx b0-4: DEST PAGE OPC_GIRO 01 xx x xxx b0-2 OFFS, b3:GET/PUT, B4-5:REG(GIRO) OPC_PAIR 1 xxx xxxx b0-3 DST, b4-6 SRC"
- note removed: "Mapped to NOP, but reserved for instruction set extensions"
- note removed: "xA adds DB val to O and carries over into D"
Changed lines of the file:
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@@
 		)
 	)
-	(text "Mapped to NOP,\nbut reserved for\ninstruction set\nextensions"
+	(text "Mapped to NOP,\nbut reserved for\ninstruction set\nexJRTensions"
 		(exclude_from_sim no)
 		(at 190.5 246.38 0)
@@
 		)
 	)
-	(text "                Instruction byte:\nall0: OPC_SYS       00000   xxx    See table @ SYS decoder\nelse: opc_RFIX       00001  x xx    b0-1 LSB, b2: Extended sign bit\n      OPC_ALU       0001   xxxx    See table @ ALU\n      OPC_TRAP      001   xxxxx    b0-4: DEST PAGE\n      OPC_GIRO      01 xx x xxx    b0-2 OFFS, b3:GET/PUT, B4-5:REG(GIRO)\n      OPC_PAIR      1  xxx xxxx    b0-3 DST, b4-6 SRC"
+	(text "                Instruction byte:\nall0: OPC_SYS       00000   xxx    See table @ SYS decoder\nelse: opc_RFIX       00001  x xx    b0-1 LSB, b2: ExJRTended sign bit\n      OPC_ALU       0001   xxxx    See table @ ALU\n      OPC_TRAP      001   xxxxx    b0-4: DEST PAGE\n      OPC_GIRO      01 xx x xxx    b0-2 OFFS, b3:GET/PUT, B4-5:REG(GIRO)\n      OPC_PAIR      1  xxx xxxx    b0-3 DST, b4-6 SRC"
 		(exclude_from_sim no)
 		(at 146.05 571.5 0)
@@
 		)
 	)
-	(text "xA adds DB val to O\nand carries over into D"
+	(text "xSKIP adds DB val to O\nand carries over into D"
 		(exclude_from_sim no)
 		(at 796.29 392.43 0)
@@
 		)
 	)
-	(text "Else sign extend\nbit 2"
+	(text "Else sign exJRTend\nbit 2"
 		(exclude_from_sim no)
 		(at 848.36 161.29 0)
@@
 		)
 	)
-	(text " 8 AND (R:=R&O)\n 9 IOR (R:=R|O)\n10 EOR (R:=R^O)\n11 ADD (Add\" / R:=R+O, bits 0-7)\n12 CAR (\"Carry Bit\" / R:= Carry, 9th bit of R+O) 00h or 01h\n13 RLO (\"Flag: R less than O\" / R:= (R<O)? 0xFF:0\n14 REO (\"Flag: R equals O\" / R:= (R==O)? 0xFF:0\n15 RGO (\"Flag: R greater than O\" / R:= (R>O)? 0xFF:0\n"
+	(text " 8 AND (R:=R&O)\n 9 IOR (R:=R|O)\n10 EOR (R:=R^O)\n11 ADD (Add\" / R:=R+O, bits 0-7)\n12 CAR (\"Carry Bit\" / R:= Carry, 9th bit of R+O) 00h or 01h\n13 RLO (\"Flag: R less than O\" / R:= (R<O)? 0xJRFF:0\n14 REO (\"Flag: R equals O\" / R:= (R==O)? 0xJRFF:0\n15 RGO (\"Flag: R greater than O\" / R:= (R>O)? 0xJRFF:0\n"
 		(exclude_from_sim no)
 		(at 1053.846 418.084 0)
@@
 		)
 	)
-	(label "Nx"
+	(label "FETCHx"
 		(at 1127.76 709.93 0)
 		(fields_autoplaced yes)
@@
 		)
 	)
-	(label "~{Nx}"
+	(label "~{FETCHx}"
 		(at 697.23 317.5 180)
 		(fields_autoplaced yes)
@@
 		)
 	)
-	(label "xT"
+	(label "xJRT"
 		(at 63.5 196.85 180)
 		(fields_autoplaced yes)
@@
 		)
 	)
-	(label "xW"
+	(label "xJWIT"
 		(at 745.49 125.73 180)
 		(fields_autoplaced yes)
@@
 		)
 	)
-	(label "xA"
+	(label "xSKIP"
 		(at 364.49 304.8 0)
 		(fields_autoplaced yes)
@@
 		)
 	)
-	(label "xJ"
+	(label "xJMP"
 		(at 63.5 194.31 180)
 		(fields_autoplaced yes)
@@
 		)
 	)
-	(label "xJ"
+	(label "xJMP"
 		(at 364.49 309.88 0)
 		(fields_autoplaced yes)
@@
 		)
 	)
-	(label "xW_pre"
+	(label "xJWIT_pre"
 		(at 63.5 191.77 180)
 		(fields_autoplaced yes)
@@
 		)
 	)
-	(label "Nx"
+	(label "FETCHx"
 		(at 712.47 317.5 0)
 		(fields_autoplaced yes)
@@
 		)
 	)
-	(label "xA"
+	(label "xSKIP"
 		(at 889 374.65 180)
 		(fields_autoplaced yes)
@@
 		)
 	)
-	(label "xC"
+	(label "xCALL"
 		(at 364.49 320.04 0)
 		(fields_autoplaced yes)
@@
 		)
 	)
-	(label "xC"
+	(label "xCALL"
 		(at 358.14 182.88 180)
 		(fields_autoplaced yes)
@@
 		)
 	)
-	(label "Nx_pre"
+	(label "FETCHx_pre"
 		(at 203.2 276.86 180)
 		(fields_autoplaced yes)
@@
 		)
 	)
-	(label "~{xW}"
+	(label "~{xJWIT}"
 		(at 760.73 125.73 0)
 		(fields_autoplaced yes)
@@
 		)
 	)
-	(label "Nx_pre"
+	(label "FETCHx_pre"
 		(at 251.46 284.48 180)
 		(fields_autoplaced yes)
@@
 		)
 	)
-	(label "Nx_pre_clean"
+	(label "FETCHx_pre_clean"
 		(at 675.64 554.99 180)
 		(fields_autoplaced yes)
@@
 		)
 	)
-	(label "xW_pre"
+	(label "xJWIT_pre"
 		(at 132.08 269.24 0)
 		(fields_autoplaced yes)
@@
 		)
 	)
-	(label "xT"
+	(label "xJRT"
 		(at 364.49 314.96 0)
 		(fields_autoplaced yes)
@@
 		)
 	)
-	(label "xA"
+	(label "xSKIP"
 		(at 854.71 317.5 180)
 		(fields_autoplaced yes)
@@
 		)
 	)
-	(label "xF"
+	(label "xJRF"
 		(at 364.49 317.5 0)
 		(fields_autoplaced yes)
@@
 		)
 	)
-	(label "~{xW}"
+	(label "~{xJWIT}"
 		(at 557.53 168.91 180)
 		(fields_autoplaced yes)
@@
 		)
 	)
-	(label "xA"
+	(label "xSKIP"
 		(at 854.71 374.65 180)
 		(fields_autoplaced yes)
@@
 		)
 	)
-	(label "~{Nx}"
+	(label "~{FETCHx}"
 		(at 361.95 373.38 0)
 		(fields_autoplaced yes)
@@
 		)
 	)
-	(label "xW"
+	(label "xJWIT"
 		(at 364.49 312.42 0)
 		(fields_autoplaced yes)
@@
 		)
 	)
-	(label "xF"
+	(label "xJRF"
 		(at 63.5 199.39 180)
 		(fields_autoplaced yes)
@@
 		)
 	)
-	(label "Nx_pre"
+	(label "FETCHx_pre"
 		(at 137.16 377.19 0)
 		(fields_autoplaced yes)
@@
 		)
 	)
-	(label "Nx_pre_clean"
+	(label "FETCHx_pre_clean"
 		(at 270.51 289.56 180)
 		(fields_autoplaced yes)
