File: Schematics/old/myth.kicad_sch (KiCad schematic)
At the start: 140 parts, among them J1 Conn_01x08_Male, J10 Conn_02x01, J2 Conn_01x08_Male, J3 Conn_01x08_Male, J4 Conn_01x08_Male, J5 Conn_01x08_Male, J6 Conn_01x08_Male, J7 Conn_01x08_Male, J8 Conn_01x04_Male, J9 Conn_01x04_Male, U1 74AHC02, U10 74HC595, U11 74HC165, U12 74AHC08, U13 74HC238, U14 74HC238, U15 74HC238, U16 4002, U17 74AHC273, U18 74LS32, U19 CD4532BE, U2 74AHC04, U20 74AHC138, U21 74AHC04, U22 74AHC138, U23 74HC238, U24 74HC238, U25 74LS32, U26 4078, U27 74AHC244, U28 74LS08, U29 74HC238, U3 74HC74, U30 74HC238, U31 4075, U32 74AHC04, U33 74HC00, U34 74HC163, U35 74AHC138, U36 74AHC138, U37 74HC238, U38 74AHC138, U39 74HC238, U4 74HC32, U40 74AHC02, U41 74AHC574, U42 74HC283, U43 74HC283, U44 74AHC574, U45 74HC193, U46 74HC193, U47 74AHC273, U49 74HC32, U5 74AHC273, U50 74AHC244, U51 74HC157, U52 74HC157, U53 74HC157, U54 74HC157, U55 74HC02, U56 74HC74, U57 74HC193, U58 74HC193, U59 74HC04, U6 74LS08, U60 4078, U61 4078, U62 74AHC574, U63 74HC193, U64 74HC193, U65 74AHC273, U66 74AHC273, U67 74LS573, U68 74LS21, U69 74AHC244, U7 74AHC08, U70 74AHC04, U71 74AHC04, U72 74LS32, U73 74AHC04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

Commit message: Let defines/labels diverge from assembler mnemonics
Parts:
- removed U60: 4078, Package_DIP:DIP-14_W7.62mm_Socket_LongPads, symbol 4xxx_IEEE:4078
- removed U8, U9: 74HC157, Package_DIP:DIP-16_W7.62mm_Socket_LongPads, symbol 74xx:74LS157
Connections:
- net FREE is gone; now on net GND: U6.10
- net IRQ0 is gone; now on net DB0: U5.3 (D0)
- net IRQ1 is gone; now on net DB1: U5.4 (D1)
- net IRQ2 is gone; now on net DB2: U5.7 (D2)
- net IRQ3 is gone; now on net DB3: U5.8 (D3)
- net IRQ4 is gone; now on net DB4: U5.13 (D4)
- net IRQ5 is gone; now on net DB5: U5.14 (D5)
- net IRQ6 is gone; now on net DB6: U5.17 (D6)
- net IRQ7 is gone; now on net DB7: U5.18 (D7)
- net +5V: now also U3.10 (~{S}), U3.13 (~{R}); no longer U3.12 (D)
- net CLOSE: no longer U59.3
- net GND: now also U2.9, U3.12 (D), U4.10, U4.9, U6.9
- net ~{PH0}: no longer U4.10
- net at U4.8: no longer U3.10 (~{S})
- net at U3.9 (Q): no longer U6.9
- net opc_RFIX renamed opc_FIX
- net xJWIT renamed xJITD
- net xJWIT_pre renamed xJITD_pre
- net xLFIX renamed xNEAR
- net xNEAR: now also U59.3; no longer U2.9
- net ~{CLOSE} renamed ~{xNEAR}
- net ~{xNEAR}: now also U45.11 (~{LOAD}), U46.11 (~{LOAD}); no longer U3.13 (~{R})
- net ~{IRQ}: no longer names the net of J4.1 (Pin_1)
- net ~{IRQ}: no longer U4.9
- net ~{opc_RFIX} renamed ~{opc_FIX}
- net ~{xJWIT} renamed ~{xJITD}
- removed net ~{xLFIX}: U2.8, U45.11 (~{LOAD}), U46.11 (~{LOAD})
- no-connect marks 66 -> 68
Other:
- note added: "FETCH-MG => END (LOX) FETCH-ML => NOP (reserved) MG-MG => NOP (reserved) MG-ML => NOP (reserved) ML-MG => NOP (reserved) ML-ML => NOP (reserved) GG => NOP (reserved) RR => NOP (reserved) II => NOP (reserved)"
- note added: "INTO DST Decoder"
- note added: "INTO SRC Decoder"
- note added: "Instruction byte: all0: OPC_SYS 00000 xxx See table @ SYS decoder else: opc_FIX 00001 x xx b0-1 LSB, b2: ExJRTended sign bit OPC_ALU 0001 xxxx See table @ ALU OPC_TRAP 001 xxxxx b0-4: DEST PAGE OPC_GIRO 01 xx x xxx b0-2 OFFS, b3:GET/PUT, B4-5:REG(GIRO) opc_PAIR 1 xxx xxxx b0-3 DST, b4-6 SRC"
- note added: "Mapped to NOP, but reserved for instruction set extensions"
- note added: "PC (the program counter) is cleared/set to 0 during TRAP or CALL. Execution starts at offset zero, the "head" of the destination page."
- note added: "Remap ("scrounge") GG, RR, II etc, and impracticable opcodes such as NM"
- note removed: "ALT: COxML7"
- note removed: "ALT: JUMP D_I"
- note removed: "ALT: RET L7_I"
- note removed: "FREE signals that code execution is outside the TRAP region (pages 0-31). Intererrupts are enabled, iff this is the case"
- note removed: "FREE signals that code execution is outside the TRAP region (pages 0-31): Intererrupts are disabled when executing within pages 0-31."
- note removed: "Instruction byte: all0: OPC_SYS 00000 xxx See table @ SYS decoder else: opc_RFIX 00001 x xx b0-1 LSB, b2: ExJRTended sign bit OPC_ALU 0001 xxxx See table @ ALU OPC_TRAP 001 xxxxx b0-4: DEST PAGE OPC_GIRO 01 xx x xxx b0-2 OFFS, b3:GET/PUT, B4-5:REG(GIRO) OPC_PAIR 1 xxx xxxx b0-3 DST, b4-6 SRC"
- note removed: "J (the program counter) is cleared/set to 0 during TRAP or CALL. Execution starts at offset zero, the "head" of the destination page."
- note removed: "MGx"
- note removed: "Mapped to NOP, but reserved for instruction set exJRTensions"
- note removed: "NM => END (LOX) NL => NOP (reserved) LM => NOP (reserved) LL => NOP (reserved) MM => NOP (reserved) ML => NOP (reserved) DD => NOP (reserved) RR => NOP (reserved) II => NOP (reserved)"
- note removed: "Pair DST Decoder"
- note removed: "Pair SRC Decoder"
- note removed: "Remap ("scrounge") DD, RR, II etc, and impracticable opcodes such as NM"
- note removed: "Selected-state output bits are a hardcoded TRAP instruction to page zero"
- note removed: "xMG"
- moved on the sheet: U18B, U18D, U2D, U3B, U4C, U6C
